File: 2_prototype_mk3/hardware/status_led.kicad_sch (KiCad schematic)
At the start: 2 parts

Commit message: Add LCSC component part numbers
Parts:
- D4: LCSC_Part_Number (none) -> C330759
- RN1: LCSC_Part_Number (none) -> C136828
Changed lines of the file:
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@@
 			)
 		)
-		(property "LCSC_Part_Number" ""
+		(property "LCSC_Part_Number" "C330759"
 			(at 132.08 90.17 0)
 			(effects
@@
 			)
 		)
-		(property "LCSC_Part_Number" ""
+		(property "LCSC_Part_Number" "C136828"
 			(at 149.86 90.17 90)
 			(effects
