File: 2_prototype_mk3/hardware/power_management.kicad_sch (KiCad schematic)
At the start: 5 parts

Commit message: MKIII design refinements
Other:
- note removed: "Ensure charging resistors is suitable for current"
- title: (none) -> Power management
- moved on the sheet: D3, D6, H3, R3, Super_Cap2

Commit message: Add net classes for power
Other:
- note added: "ISA bus power For ISA slot mode"
- title: Power management -> (none)
- moved on the sheet: D3, D6, H3, R3, Super_Cap2

Commit message: MKIII PCB components connected and passing DRC
Connections:
- net VSYS_5V_INPUT renamed POWER_5V_SUP
Changed lines of the file:
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@@
+	(wire
+		(pts
+			(xy 148.59 80.01) (xy 148.59 81.28)
+		)
+		(stroke
+			(width 0)
+			(type default)
+		)
+	)
 	(wire
 		(pts
@@
 			(width 0)
 			(type default)
+		)
+	)
+	(global_label "POWER_5V_SUP"
+		(shape bidirectional)
+		(at 148.59 80.01 90)
+		(fields_autoplaced yes)
+		(effects
+			(font
+				(size 1.27 1.27)
+			)
+			(justify left)
+		)
+		(property "Intersheetrefs" "${INTERSHEET_REFS}"
+			(at 148.59 61.3993 90)
+			(effects
+				(font
+					(size 1.27 1.27)
+				)
+				(justify left)
+				(hide yes)
+			)
 		)
 	)
@@
 			(justify left bottom)
 		)
-		(property "Netclass" "POWER_5v"
+		(property "Netclass" "POWER_5V_SUP"
 			(at 158.1785 78.74 0)
 			(effects
@@
 			(effects
 				(font
+					(size 1.27 1.27)
+					(italic yes)
+				)
+			)
+		)
+	)
+	(netclass_flag ""
+		(length 2.54)
+		(shape round)
+		(at 152.4 93.98 180)
+		(fields_autoplaced yes)
+		(effects
+			(font
+				(size 1.27 1.27)
+			)
+			(justify right bottom)
+		)
+		(property "Netclass" "POWER_5V_SUP"
+			(at 153.0985 96.52 0)
+			(effects
+				(font
+					(size 1.27 1.27)
+				)
+				(justify left)
+			)
+		)
+		(property "Component Class" ""
+			(at -54.61 8.89 0)
+			(effects
+				(font

Commit message: Add manufacturer part nu bers
Parts:
- D3: Manufacturer_Part_Number (none) -> SS12
- D6: Manufacturer_Part_Number (none) -> SS14
- R3: Manufacturer_Part_Number (none) -> RC1206FR-0733RL
- Super_Cap2: Manufacturer_Part_Number (none) -> DX-5R5V474U
Changed lines of the file:
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@@
+			)
+		)
+		(property "Manufacturer_Part_Number" "SS12"
+			(at 142.24 90.17 90)
+			(effects
+				(font
+					(size 1.27 1.27)
+				)
+				(hide yes)
 			)
 		)
@@
 			)
 		)
+		(property "Manufacturer_Part_Number" "SS14"
+			(at 189.23 90.17 0)
+			(effects
+				(font
+					(size 1.27 1.27)
+				)
+				(hide yes)
+			)
+		)
 		(pin "2"
 		)
@@
 		)
 		(property "Description" "Unpolarized capacitor, small symbol"
+			(at 148.59 96.52 0)
+			(effects
+				(font
+					(size 1.27 1.27)
+				)
+				(hide yes)
+			)
+		)
+		(property "Manufacturer_Part_Number" "DX-5R5V474U"
 			(at 148.59 96.52 0)
 			(effects
@@
 			)
 		)
+		(property "Manufacturer_Part_Number" "RC1206FR-0733RL"
+			(at 154.94 90.17 0)
+			(effects
+				(font
+					(size 1.27 1.27)
+				)
+				(hide yes)
+			)
+		)
 		(pin "1"
 		)
@@
 			(at 114.3 93.98 0)
 			(effects
+				(font
+					(size 1.27 1.27)
+				)
+				(hide yes)
+			)
+		)
+		(property "Manufacturer_Part_Number" ""
+			(at 114.3 93.98 0)
+			(effects

Commit message: Switch SD card reader to better component
Parts:
- H3: now not fitted
Changed lines of the file:
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@@
 		(in_bom yes)
 		(on_board yes)
-		(dnp no)
+		(dnp yes)
 		(property "Reference" "H3"
 			(at 115.57 85.09 0)
