File: 2_prototype_mk3/hardware/power_management.kicad_sch (KiCad schematic)
At the start: 5 parts

Commit message: Add LCSC components part numbers
Parts:
- D3: LCSC_Part_Number (none) -> C184027
- D6: LCSC_Part_Number (none) -> C83852
Changed lines of the file:
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@@
+			)
+		)
+		(property "LCSC_Part_Number" "C184027"
+			(at 142.24 90.17 90)
+			(effects
+				(font
+					(size 1.27 1.27)
+				)
+				(hide yes)
 			)
 		)
@@
 			)
 		)
+		(property "LCSC_Part_Number" "C83852"
+			(at 189.23 90.17 0)
+			(effects
+				(font
+					(size 1.27 1.27)
+				)
+				(hide yes)
+			)
+		)
 		(pin "2"
 		)
@@
 		)
 		(property "Manufacturer" ""
+			(at 148.59 96.52 0)
+			(effects
+				(font
+					(size 1.27 1.27)
+				)
+				(hide yes)
+			)
+		)
+		(property "LCSC_Part_Number" ""
 			(at 148.59 96.52 0)
 			(effects
@@
 			)
 		)
+		(property "LCSC_Part_Number" ""
+			(at 154.94 90.17 0)
+			(effects
+				(font
+					(size 1.27 1.27)
+				)
+				(hide yes)
+			)
+		)
 		(pin "1"
 		)
@@
 			(at 114.3 93.98 0)
 			(effects
+				(font
+					(size 1.27 1.27)
+				)
+				(hide yes)
+			)
+		)
+		(property "LCSC_Part_Number" ""
+			(at 114.3 93.98 0)
+			(effects
