File: 2_prototype_mk3/hardware/amplifier.kicad_sch (KiCad schematic)
At the start: 8 parts, among them U5 MAX98357A

Commit message: Add LCSC components part numbers
Parts:
- FB1, FB2: LCSC_Part_Number (none) -> C85840
- H6: LCSC_Part_Number (none) -> C3819527
- U5: LCSC_Part_Number (none) -> C910544
Changed lines of the file:
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@@
+			)
+		)
+		(property "LCSC_Part_Number" ""
+			(at 195.58 115.57 0)
+			(effects
+				(font
+					(size 1.27 1.27)
+				)
+				(hide yes)
 			)
 		)
@@
 			)
 		)
+		(property "LCSC_Part_Number" "C3819527"
+			(at 212.09 106.68 0)
+			(effects
+				(font
+					(size 1.27 1.27)
+				)
+				(hide yes)
+			)
+		)
 		(pin "1"
 		)
@@
 			)
 		)
+		(property "LCSC_Part_Number" ""
+			(at 143.51 64.77 0)
+			(effects
+				(font
+					(size 1.27 1.27)
+				)
+				(hide yes)
+			)
+		)
 		(pin "2"
 		)
@@
 		)
 		(property "Manufacturer" ""
+			(at 160.02 64.77 0)
+			(effects
+				(font
+					(size 1.27 1.27)
+				)
+				(hide yes)
+			)
+		)
+		(property "LCSC_Part_Number" ""
 			(at 160.02 64.77 0)
 			(effects
@@
 			)
 		)
+		(property "LCSC_Part_Number" "C910544"
+			(at 149.86 105.41 0)
+			(effects
+				(font
+					(size 1.27 1.27)
+				)
+				(hide yes)
+			)
+		)
 		(pin "16"
 		)
@@
 			)
 		)
+		(property "LCSC_Part_Number" "C85840"
+			(at 181.61 101.6 0)
+			(effects
+				(font
+					(size 1.27 1.27)
+				)
+				(hide yes)
+			)
+		)
 		(pin "1"
 		)
@@
 			)
 		)
+		(property "LCSC_Part_Number" ""
+			(at 204.47 115.57 0)
+			(effects
+				(font
+					(size 1.27 1.27)
+				)
+				(hide yes)
+			)
+		)
 		(pin "1"
 		)
@@
 			(at 172.72 106.68 0)
 			(effects
+				(font
+					(size 1.27 1.27)
+				)
+				(hide yes)
+			)
+		)
+		(property "LCSC_Part_Number" "C85840"
+			(at 172.72 106.68 0)
+			(effects
