File: 2_prototype_mk3/hardware/sdcard_reader.kicad_sch (KiCad schematic)
At the start: 4 parts, among them J1 Micro_SD_Card

Commit message: Add LCSC component part numbers
Parts:
- RN2: LCSC_Part_Number (none) -> C779384
Changed lines of the file:
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@@
 			)
 		)
-		(property "LCSC_Part_Number" ""
+		(property "LCSC_Part_Number" "C779384"
 			(at 88.9 77.47 0)
 			(effects
