File: 2_prototype_mk4/hardware/oled.kicad_sch (KiCad schematic)
At the start: 1 part, among them J7 Conn_01x04_Pin

Commit message: MK4 PCB layout complete
Other:
- note added: "OLED screen header (Optional) 1) VCC 3.3V 2) GND GND pin 3) SCL I2C SCL pin 4) SDA I2C SDA Pin"
- note removed: "OLED screen debug output 1) VCC 3.3V 2) GND GND pin 3) SCL I2C SCL pin 4) SDA I2C SDA Pin"
Changed lines of the file:
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@@
 	(generator_version "10.0")
 	(paper "A4")
-	(text "OLED screen debug output\n\n1) VCC	3.3V\n2) GND	GND pin\n3) SCL	I2C SCL pin\n4) SDA	I2C SDA Pin"
+	(text "OLED screen header (Optional)\n\n1) VCC	3.3V\n2) GND	GND pin\n3) SCL	I2C SCL pin\n4) SDA	I2C SDA Pin"
 		(exclude_from_sim no)
 		(at 148.59 84.328 0)
