File: 2_prototype_mk4/hardware/rotary_encoder.kicad_sch (KiCad schematic)
At the start: 2 parts, among them J8 Conn_01x05, SW2 PEC12R-2120F-S0012

Commit message: MK4 PCB layout complete
Other:
- note added: "Volume/balance encoder header (Optional)"
- note removed: "An optional component in the MKIV"
Changed lines of the file:
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@@
 		)
 	)
-	(text "An optional component in the MKIV"
+	(text "Volume/balance encoder header (Optional)"
 		(exclude_from_sim no)
 		(at 194.31 71.12 0)

Commit message: Update MKIV hardware & use MKIII software as basic for MKIV
Parts:
- SW2: Manufacturer Bourns -> (none)
Changed lines of the file:
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@@
-			)
-		)
-		(property "Manufacturer" "Bourns"
-			(at 146.05 77.47 0)
-			(hide yes)
-			(show_name no)
-			(do_not_autoplace no)
-			(effects
-				(font
-					(size 1.27 1.27)
-				)
 			)
 		)
