File: 2_prototype_mk4/hardware/sdcard_reader.kicad_sch (KiCad schematic)
At the start: 4 parts, among them J1 Micro_SD_Card

Commit message: Update MKIV hardware & use MKIII software as basic for MKIV
Parts:
- J1: Manufacturer Hirose Electric -> (none)
Changed lines of the file:
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@@
-			)
-		)
-		(property "Manufacturer" ""
-			(at 88.9 77.47 0)
-			(hide yes)
-			(show_name no)
-			(do_not_autoplace no)
-			(effects
-				(font
-					(size 1.27 1.27)
-				)
 			)
 		)
@@
 			)
 		)
-		(property "Manufacturer" ""
-			(at 113.03 60.96 0)
-			(hide yes)
-			(show_name no)
-			(do_not_autoplace no)
-			(effects
-				(font
-					(size 1.27 1.27)
-				)
-			)
-		)
 		(property "LCSC_Part_Number" ""
 			(at 113.03 60.96 0)
@@
 			)
 		)
-		(property "Manufacturer" "Hirose Electric"
-			(at 147.32 92.71 0)
-			(hide yes)
-			(show_name no)
-			(do_not_autoplace no)
-			(effects
-				(font
-					(size 1.27 1.27)
-				)
-			)
-		)
 		(property "LCSC_Part_Number" "C719027"
 			(at 147.32 92.71 0)
@@
 			(at 97.79 60.96 0)
 			(hide yes)
-			(show_name no)
-			(do_not_autoplace no)
-			(effects
-				(font
-					(size 1.27 1.27)
-				)
-			)
-		)
-		(property "Manufacturer" ""
-			(at 97.79 60.96 0)
-			(hide yes)
