File: 2_prototype_mk4/hardware/amplifier.kicad_sch (KiCad schematic)
At the start: 8 parts, among them U1 MAX98357A

Commit message: Update MKIV hardware & use MKIII software as basic for MKIV
Parts:
- H1: Manufacturer Phoenix Contact -> (none)
- U1: Manufacturer Analog Devices -> (none)
Changed lines of the file:
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@@
-			)
-		)
-		(property "Manufacturer" ""
-			(at 187.96 96.52 0)
-			(hide yes)
-			(show_name no)
-			(do_not_autoplace no)
-			(effects
-				(font
-					(size 1.27 1.27)
-				)
 			)
 		)
@@
 			)
 		)
-		(property "Manufacturer" "Phoenix Contact"
-			(at 212.09 100.33 0)
-			(hide yes)
-			(show_name no)
-			(do_not_autoplace no)
-			(effects
-				(font
-					(size 1.27 1.27)
-				)
-			)
-		)
 		(property "LCSC_Part_Number" "C3819527"
 			(at 212.09 100.33 0)
@@
 			)
 		)
-		(property "Manufacturer" ""
-			(at 143.51 64.77 0)
-			(hide yes)
-			(show_name no)
-			(do_not_autoplace no)
-			(effects
-				(font
-					(size 1.27 1.27)
-				)
-			)
-		)
 		(property "LCSC_Part_Number" ""
 			(at 143.51 64.77 0)
@@
 		)
 		(property "Manufacturer_Part_Number" "CL31A106KAHNNNE"
-			(at 160.02 64.77 0)
-			(hide yes)
-			(show_name no)
-			(do_not_autoplace no)
-			(effects
-				(font
-					(size 1.27 1.27)
-				)
-			)
-		)
-		(property "Manufacturer" ""
 			(at 160.02 64.77 0)
 			(hide yes)
@@
 			)
 		)
-		(property "Manufacturer" "Analog Devices"
-			(at 149.86 105.41 0)
-			(hide yes)
-			(show_name no)
-			(do_not_autoplace no)
-			(effects
-				(font
-					(size 1.27 1.27)
-				)
-			)
-		)
 		(property "LCSC_Part_Number" "C910544"
 			(at 149.86 105.41 0)
@@
 			)
 		)
-		(property "Manufacturer" ""
-			(at 177.8 91.44 0)
-			(hide yes)
-			(show_name no)
-			(do_not_autoplace no)
-			(effects
-				(font
-					(size 1.27 1.27)
-				)
-			)
-		)
 		(property "LCSC_Part_Number" "C85840"
 			(at 177.8 91.44 0)
@@
 			)
 		)
-		(property "Manufacturer" ""
-			(at 193.04 101.6 0)
-			(hide yes)
-			(show_name no)
-			(do_not_autoplace no)
-			(effects
-				(font
-					(size 1.27 1.27)
-				)
-			)
-		)
 		(property "LCSC_Part_Number" ""
 			(at 193.04 101.6 0)
@@
 			(at 177.8 106.68 0)
 			(hide yes)
-			(show_name no)
-			(do_not_autoplace no)
-			(effects
-				(font
-					(size 1.27 1.27)
-				)
-			)
-		)
-		(property "Manufacturer" ""
-			(at 177.8 106.68 0)
-			(hide yes)

Commit message: Final MKIV tweaks before sending off to PCBWay
Connections:
- net POWER_5V_SUP: no longer U1.4 (~{SD_MODE})
- new net SD_MODE: U1.4 (~{SD_MODE})
Changed lines of the file:
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@@
 	(text "Connect to GND: 9dB gain (Quiet/Cleanest).\nConnect to VDD (5V): 12dB gain (Standard).\nConnect to VDD through a 100kOhm resistor: 15dB (Loud).\nLeave Floating (Unconnected): 6dB (Very quiet)."
 		(exclude_from_sim no)
-		(at 77.724 117.602 0)
+		(at 71.882 121.158 0)
 		(effects
 			(font
@@
 	)
 	(junction
-		(at 132.08 107.95)
-		(diameter 0)
-		(color 0 0 0 0)
-	)
-	(junction
 		(at 187.96 91.44)
 		(diameter 0)
@@
 	(wire
 		(pts
-			(xy 132.08 110.49) (xy 137.16 110.49)
-		)
-		(stroke
-			(width 0)
-			(type default)
-		)
-	)
-	(wire
-		(pts
 			(xy 147.32 120.65) (xy 147.32 124.46)
 		)
@@
 	(wire
 		(pts
+			(xy 118.11 107.95) (xy 137.16 107.95)
+		)
+		(stroke
+			(width 0)
+			(type default)
+		)
+	)
+	(wire
+		(pts
 			(xy 165.1 100.33) (xy 165.1 106.68)
 		)
@@
 	(wire
 		(pts
-			(xy 132.08 107.95) (xy 132.08 110.49)
-		)
-		(stroke
-			(width 0)
-			(type default)
-		)
-	)
-	(wire
-		(pts
 			(xy 149.86 55.88) (xy 149.86 60.96)
 		)
@@
 	(wire
 		(pts
-			(xy 132.08 107.95) (xy 137.16 107.95)
-		)
-		(stroke
-			(width 0)
-			(type default)
-		)
-	)
-	(wire
-		(pts
 			(xy 165.1 97.79) (xy 162.56 97.79)
 		)
@@
 	(wire
 		(pts
-			(xy 121.92 107.95) (xy 132.08 107.95)
+			(xy 121.92 110.49) (xy 137.16 110.49)
 		)
 		(stroke
@@
 	(global_label "POWER_5V_SUP"
 		(shape bidirectional)
-		(at 121.92 107.95 180)
+		(at 121.92 110.49 180)
 		(fields_autoplaced yes)
 		(effects
@@
 		)
 		(property "Intersheetrefs" "${INTERSHEET_REFS}"
-			(at 103.3093 107.95 0)
+			(at 103.3093 110.49 0)
 			(hide yes)
 			(show_name no)
@@
 		)
 	)
+	(hierarchical_label "SD_MODE"
+		(shape input)
+		(at 118.11 107.95 180)
+		(effects
+			(font
+				(size 1.27 1.27)
+			)
+			(justify right)
+		)
+	)
 	(hierarchical_label "BCLK"
 		(shape input)
@@
 		(length 2.54)
 		(shape round)
-		(at 127 107.95 0)
+		(at 127 110.49 180)
 		(fields_autoplaced yes)
 		(effects
@@
 				(size 1.27 1.27)
 			)
-			(justify left bottom)
+			(justify right bottom)
 		)
 		(property "Net Class" "Power"
-			(at 127.6985 105.41 0)
+			(at 127.6985 113.03 0)
 			(show_name no)
 			(do_not_autoplace no)
@@
 		)
 		(property "Component Class" ""
-			(at -46.99 13.97 0)
+			(at -46.99 16.51 0)
 			(show_name no)
 			(do_not_autoplace no)
