File: 2_prototype_mk5/hardware/reset.kicad_sch (KiCad schematic)
At the start: 5 parts, among them Q1 2N7002

Commit message: Major MKV redesign using embedded RP2350
Parts:
- renumbered C9 to C26, D5 to D3, H9 to H13, R10 to R17
Changed lines of the file:
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@@
 		(dnp no)
 		(fields_autoplaced yes)
-		(property "Reference" "R10"
+		(property "Reference" "R17"
 			(at 148.59 113.0299 0)
 			(show_name no)
@@
 			(project "HDD Synth Prototype MK5"
 				(path "/1a22431a-ba36-40a0-9a7e-c2a82ec69c53/793258e2-de63-4f09-86a3-fe48790268bf"
-					(reference "R10")
+					(reference "R17")
 					(unit 1)
 				)
@@
 		(dnp no)
 		(fields_autoplaced yes)
-		(property "Reference" "C9"
+		(property "Reference" "C26"
 			(at 142.24 96.5201 0)
 			(show_name no)
@@
 			(project "HDD Synth Prototype MK5"
 				(path "/1a22431a-ba36-40a0-9a7e-c2a82ec69c53/793258e2-de63-4f09-86a3-fe48790268bf"
-					(reference "C9")
+					(reference "C26")
 					(unit 1)
 				)
@@
 		(dnp no)
 		(fields_autoplaced yes)
-		(property "Reference" "#PWR033"
+		(property "Reference" "#PWR052"
 			(at 146.05 128.27 0)
 			(hide yes)
@@
 			(project "HDD Synth Prototype MK5"
 				(path "/1a22431a-ba36-40a0-9a7e-c2a82ec69c53/793258e2-de63-4f09-86a3-fe48790268bf"
-					(reference "#PWR033")
+					(reference "#PWR052")
 					(unit 1)
 				)
@@
 		(dnp no)
 		(fields_autoplaced yes)
-		(property "Reference" "#PWR017"
+		(property "Reference" "#PWR051"
 			(at 146.05 88.9 0)
 			(hide yes)
@@
 			(project "HDD Synth Prototype MK5"
 				(path "/1a22431a-ba36-40a0-9a7e-c2a82ec69c53/793258e2-de63-4f09-86a3-fe48790268bf"
-					(reference "#PWR017")
+					(reference "#PWR051")
 					(unit 1)
 				)
@@
 		(dnp no)
 		(fields_autoplaced yes)
-		(property "Reference" "H9"
+		(property "Reference" "H13"
 			(at 204.47 93.9799 90)
 			(show_name no)
@@
 			(project "HDD Synth Prototype MK5"
 				(path "/1a22431a-ba36-40a0-9a7e-c2a82ec69c53/793258e2-de63-4f09-86a3-fe48790268bf"
-					(reference "H9")
+					(reference "H13")
 					(unit 1)
 				)
@@
 		(dnp no)
 		(fields_autoplaced yes)
-		(property "Reference" "#PWR038"
+		(property "Reference" "#PWR053"
 			(at 162.56 128.27 0)
 			(hide yes)
@@
 			(project "HDD Synth Prototype MK5"
 				(path "/1a22431a-ba36-40a0-9a7e-c2a82ec69c53/793258e2-de63-4f09-86a3-fe48790268bf"
-					(reference "#PWR038")
+					(reference "#PWR053")
 					(unit 1)
 				)
@@
 		(dnp no)
 		(fields_autoplaced yes)
-		(property "Reference" "#PWR036"
+		(property "Reference" "#PWR054"
 			(at 180.34 128.27 0)
 			(hide yes)
@@
 			(project "HDD Synth Prototype MK5"
 				(path "/1a22431a-ba36-40a0-9a7e-c2a82ec69c53/793258e2-de63-4f09-86a3-fe48790268bf"
-					(reference "#PWR036")
+					(reference "#PWR054")
 					(unit 1)
 				)
@@
 		(dnp no)
 		(fields_autoplaced yes)
-		(property "Reference" "D5"
+		(property "Reference" "D3"
 			(at 165.1 113.0299 90)
 			(show_name no)
@@
 			(project "HDD Synth Prototype MK5"
 				(path "/1a22431a-ba36-40a0-9a7e-c2a82ec69c53/793258e2-de63-4f09-86a3-fe48790268bf"
-					(reference "D5")
-					(unit 1)
-				)
+					(reference "D3")
+					(unit 1)
+				)

Commit message: MKV: Add LCSC numbers and resolve DRC errors
Parts:
- C26: LCSC_Part_Number (none) -> C14663
- D3: LCSC_Part_Number (none) -> C81598
- H13: LCSC_Part_Number (none) -> C124375
- Q1: LCSC_Part_Number (none) -> C332103
- R17: LCSC_Part_Number (none) -> C60491
