File: 2_prototype_mk5/hardware/reset.kicad_sch (KiCad schematic)
At the start: 5 parts, among them Q1 2N7002

Commit message: MKV revision 1
Parts:
- C26: LCSC Part Number (none) -> C14663; LCSC_Part_Number C14663 -> (none)
- D3: LCSC Part Number (none) -> C81598; LCSC_Part_Number C81598 -> (none)
- H13: LCSC Part Number (none) -> C124375; LCSC_Part_Number C124375 -> (none)
- Q1: LCSC Part Number (none) -> C332103; LCSC_Part_Number C332103 -> (none)
- R17: LCSC Part Number (none) -> C60491; LCSC_Part_Number C60491 -> (none)
Changed lines of the file:
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@@
 			)
 		)
-		(property "LCSC_Part_Number" "C60491"
+		(property "LCSC Part Number" "C60491"
 			(at 146.05 114.3 0)
 			(hide yes)
@@
 			)
 		)
-		(property "LCSC_Part_Number" "C14663"
-			(at 146.05 95.25 0)
-			(hide yes)
-			(show_name no)
-			(do_not_autoplace no)
-			(effects
-				(font
-					(size 1.27 1.27)
-				)
-			)
-		)
 		(property "Availability" ""
 			(at 146.05 95.25 0)
@@
 		)
 		(property "SnapEDA_Link" ""
+			(at 146.05 95.25 0)
+			(hide yes)
+			(show_name no)
+			(do_not_autoplace no)
+			(effects
+				(font
+					(size 1.27 1.27)
+				)
+			)
+		)
+		(property "LCSC Part Number" "C14663"
 			(at 146.05 95.25 0)
 			(hide yes)
@@
 			)
 		)
-		(property "LCSC_Part_Number" "C124375"
-			(at 201.93 95.25 0)
-			(hide yes)
-			(show_name no)
-			(do_not_autoplace no)
-			(effects
-				(font
-					(size 1.27 1.27)
-				)
-			)
-		)
 		(property "Availability" ""
 			(at 201.93 95.25 90)
@@
 		)
 		(property "SnapEDA_Link" ""
+			(at 201.93 95.25 90)
+			(hide yes)
+			(show_name no)
+			(do_not_autoplace no)
+			(effects
+				(font
+					(size 1.27 1.27)
+				)
+			)
+		)
+		(property "LCSC Part Number" "C124375"
 			(at 201.93 95.25 90)
 			(hide yes)
@@
 			)
 		)
-		(property "LCSC_Part_Number" "C81598"
+		(property "LCSC Part Number" "C81598"
 			(at 162.56 114.3 90)
 			(hide yes)
@@
 			)
 		)
-		(property "LCSC_Part_Number" "C332103"
-			(at 177.8 104.14 0)
-			(hide yes)
+		(property "LCSC Part Number" "C332103"
+			(at 177.8 104.14 0)
+			(hide yes)

Commit message: Add buck boost to 5V and reset line stability
Parts:
- added R23: 10K, Resistor_SMD:R_0402_1005Metric, symbol Device:R
- added R26: 1K, Resistor_SMD:R_0402_1005Metric, symbol Device:R
Connections:
- net at D3.1 (K), Q1.1 (G), R17.1: now also R23.2; no longer C26.1
- net at Q1.3 (D): now also R26.1; no longer H13.2 (Pin_2)
- new net: C26.1, R23.1
- new net: H13.2 (Pin_2), R26.2
Other:
- moved on the sheet: C26

Commit message: Cost reductions for JCLPCB
Parts:
- H13: now not fitted; now left out of the parts list
- Q1: LCSC Part Number C332103 -> C8545
- R17: LCSC Part Number C60491 -> C25741
- R23: LCSC Part Number (none) -> C25744
- R26: LCSC Part Number (none) -> C11702
Changed lines of the file:
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@@
 			)
 		)
-		(property "LCSC Part Number" "C60491"
+		(property "LCSC Part Number" "C25741"
 			(at 146.05 114.3 0)
 			(hide yes)
@@
 			)
 		)
-		(property "LCSC Part Number" ""
+		(property "LCSC Part Number" "C11702"
 			(at 189.23 90.17 0)
 			(hide yes)
@@
 		(body_style 1)
 		(exclude_from_sim no)
-		(in_bom yes)
+		(in_bom no)
 		(on_board yes)
 		(in_pos_files yes)
-		(dnp no)
+		(dnp yes)
 		(fields_autoplaced yes)
 		(property "Reference" "H13"
@@
 			)
 		)
-		(property "LCSC Part Number" ""
+		(property "LCSC Part Number" "C25744"
 			(at 146.05 95.25 0)
 			(hide yes)
@@
 			)
 		)
-		(property "LCSC Part Number" "C332103"
+		(property "LCSC Part Number" "C8545"
 			(at 177.8 104.14 0)
 			(hide yes)
