File: 2_prototype_mk5/hardware/HDD Synth Prototype MK5.kicad_pcb (KiCad board)
At the start: 2 copper layers, 100.3 x 69.9 mm, 83 parts, among them J1 Micro_SD_Card, J2 Conn_01x03, J4 USB_C_Receptacle_USB2.0_16P, J6 Conn_01x04_Pin, J7 Conn_01x05, Q1 2N7002, SW1 SW_Push, SW2 SW_Push, U1 Optocoupler_DC_PhotoNPN_AKEC, U2 MAX98357A, U3 W25Q128JVS, U4 NCP1117-3.3_SOT223, U5 RP2350_60QFN, Y1 ABM8-272-T3

Commit message: Successful MKV software test (after minor modification)
Parts:
- removed SW1, SW2: SW_Push, Button_Switch_SMD:SW_Push_1P1T_NO_Vertical_Wuerth_434133025816
- added S1: TS-1187A-B-A-B, Custom:SW_TS-1187A-B-A-B, F.Cu at (131.6, 113.6)
- added S2: TS-1187A-B-A-B, Custom:SW_TS-1187A-B-A-B, F.Cu at (168.1, 60.3)
- C10, C14, C17, C18, C19, C20, C21, C22, C23, C24: value 100n -> 100nF
- C11, C25, C9: value 10u -> 10uF
- C12, C13, C15, C16: value 4.7u -> 4.7uF
- J4: footprint Connector_USB:USB_C_Receptacle_Amphenol_12401610E4-2A -> Connector_USB:USB_C_Receptacle_HRO_TYPE-C-31-M-12
- R13: value 33 -> 33R
- R15, R16: value 27 -> 27R
- R5: value 33R -> 47R
- moved R12 12.1 mm to (124.0, 115.6), turned to 180 degrees
- moved R11 3.43 mm to (162.1, 68.6)
- moved J4 1.09 mm to (168.9, 71.6)
- moved R8 0.72 mm to (162.1, 73.7)
Routing:
- net +3V3: track 221.3 -> 200.8 mm
- net /RP2350/~{USB_BOOT}: track 21.5 -> 28.3 mm, vias 0 -> 2
- net Net-(J4-CC2): track 8.73 -> 2.84 mm, vias 2 -> 0
- net Net-(R12-Pad1): track 6.69 -> 10.2 mm
- net GND: track 121.7 -> 125.2 mm
- net /RP2350/USB_D+: track 11.4 -> 12.2 mm, vias 2 -> 0
- net /RP2350/RUN: track 51.6 -> 52.3 mm
- net /RP2350/USB_D-: track 12.7 -> 12.5 mm, vias 2 -> 0

Commit message: MKV revision 1
Parts:
- removed C27: 0.1uF, Capacitor_SMD:C_0603_1608Metric
- removed D4: WS2812B, LED_SMD:LED_WS2812B_PLCC4_5.0x5.0mm_P3.2mm
- removed H4, H5, H6, H7: MountingHole, MountingHole:MountingHole_3.2mm_M3
- added H14: Conn_01x02, Connector_PinHeader_2.54mm:PinHeader_1x02_P2.54mm_Vertical, F.Cu at (167.6, 110.5)
- added LED1: XL-3528RGBW-HM, Custom:LED-SMD_4P-L3.2-W2.8-LS3.5-XL-3528RGBW-HM5, F.Cu at (168.6, 54.1)
- added R18: 56R, Resistor_SMD:R_0402_1005Metric, F.Cu at (165.9, 49.5)
- added R19: 270R, Resistor_SMD:R_0402_1005Metric, F.Cu at (165.9, 50.8)
- added R20: 33R, Resistor_SMD:R_0402_1005Metric, F.Cu at (165.9, 48.3)
- R5: value 47R -> 22R
- U3: value W25Q128JVS -> W25Q32JVSSIQ
- moved R2 8.10 mm to (137.6, 98.6), turned to -90 degrees
- moved J2 5.08 mm to (120.7, 74.0), turned to 90 degrees
- moved H12 2.83 mm to (110.3, 58.4)
- moved FB1 2.62 mm to (116.7, 62.2)
- moved FB2 2.62 mm to (116.7, 58.4)
- moved H13 2.41 mm to (130.8, 107.4), turned to 90 degrees
- moved H3 2.41 mm to (130.8, 99.1), turned to 90 degrees
- moved H1 2.41 mm to (120.7, 107.4), turned to 90 degrees
- moved H2 2.41 mm to (120.7, 99.1), turned to 90 degrees
- moved C1 2.39 mm to (123.8, 66.3)
- moved C2 2.39 mm to (126.3, 64.0)
- moved C3 2.39 mm to (120.5, 64.8)
- moved C4 2.39 mm to (120.5, 55.9)
- moved U2 2.39 mm to (125.0, 59.2)
- moved J1 2.17 mm to (139.6, 57.1), turned to 180 degrees
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Connections:
- U5 pad 7: /RP2350/GPIO4 -> /RP2350/RGB_LED_RED
- U5 pad 8: /RP2350/GPIO5 -> /RP2350/RGB_LED_GREEN
- U5 pad 9: /RP2350/GPIO6 -> /RP2350/RBG_LED_BLUE
Routing:
- net /RP2350/LED_DATA: track 32.6 -> 0.00 mm, vias 2 -> 0
- net /RP2350/RBG_LED_BLUE: track 0.00 -> 32.3 mm, vias 0 -> 2
- net /RP2350/RGB_LED_GREEN: track 0.00 -> 30.3 mm, vias 0 -> 2
- net /RP2350/RGB_LED_RED: track 0.00 -> 29.2 mm, vias 0 -> 2
- net +5V: track 65.7 -> 81.5 mm
- net /RP2350/SD_SCK: track 12.3 -> 27.2 mm
- net Net-(LED1-B-): track 0.00 -> 14.2 mm
- net /RP2350/SD_MISO: track 37.7 -> 24.6 mm, vias 2 -> 0
- net /RP2350/SD_CS: track 24.9 -> 36.8 mm
- net /RP2350/SD_MOSI: track 24.2 -> 35.6 mm, vias 2 -> 0
- net POWER_5V_SUP: track 155.3 -> 144.4 mm
- net /RP2350/SWD: track 27.9 -> 21.7 mm
- net /RP2350/SWCLK: track 21.3 -> 27.3 mm
- net Net-(LED1-R-): track 0.00 -> 5.62 mm
- net +3V3: track 200.8 -> 206.3 mm, vias 2 -> 4
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Other:
- outline, holes or cut-outs redrawn
- board text added: "+"
- board text added: "-"
- board text added: "Aux 5v input"
- board text added: "Revision 1"
- board text added: "SD card reader"
