File: 2_prototype_mk5/hardware/HDD Synth Prototype MK5.kicad_pcb (KiCad board)
At the start: 2 copper layers, 100.3 x 69.9 mm, 112 parts, among them J2 Conn_01x03, J4 USB_C_Receptacle_USB2.0_16P, J6 Conn_01x04_Pin, J7 Conn_01x05, Q1 2N7002, U1 Optocoupler_DC_PhotoNPN_AKEC, U2 MAX98357A, U3 W25Q32JVSSIQ, U5 RP2350_60QFN, U6 TPS63020DSJR, U7 KF350-3.5-2P, U8 TPS25921ADR, U9 TPS61094DSSR, Y1 ABM8-272-T3

Commit message: Schematics and layout complete for 5.2.0
Co-Authored-By: Claude Sonnet 5 <noreply@anthropic.com>
Parts:
- Super_Cap1: footprint Capacitor_THT:CP_Radial_D14.0mm_P5.00mm -> Custom:SuperCap_Eaton_PHV_9.0x17.3mm_P11.80mm
- moved C30 14.9 mm to (154.0, 110.5), turned to 0 degrees
- moved C27 9.67 mm to (144.3, 110.5), turned to 0 degrees
- moved C28 8.98 mm to (148.9, 110.5), turned to 0 degrees
- moved Super_Cap1 0.37 mm to (149.0, 104.1)
Routing:
- net GND: track 155.2 -> 180.7 mm, vias 55 -> 68
- net Net-(H13-Pin_2): track 0.00 -> 22.9 mm, vias 0 -> 1
- net +3V3: track 251.8 -> 273.3 mm, vias 4 -> 6
- net /RP2350/PWR_FAULT_N: track 25.5 -> 31.2 mm, vias 1 -> 2
- net VSYS: track 171.5 -> 166.9 mm
- net Net-(U9-SUP): track 58.2 -> 61.7 mm
- net /Power/VIN_PROT: track 19.0 -> 22.5 mm
Other:
- board text added: "Version 5.3.0 Beta test edition"
- board text removed: "Version 5.2.0 Beta test edition"
