File: 2_prototype_mk5/hardware/HDD Synth Prototype MK5.kicad_pcb (KiCad board)
At the start: 2 copper layers, 100.3 x 69.9 mm, 112 parts, among them J2 Conn_01x03, J4 USB_C_Receptacle_USB2.0_16P, J6 Conn_01x04_Pin, J7 Conn_01x05, Q1 2N7002, U1 Optocoupler_DC_PhotoNPN_AKEC, U2 MAX98357A, U3 W25Q32JVSSIQ, U5 RP2350_60QFN, U6 TPS63020DSJR, U7 KF350-3.5-2P, U8 TPS25921ADR, U9 TPS61094DSSR, Y1 ABM8-272-T3

Commit message: 5.3.0 sent to JCLPCB
Parts:
- R35: value 100K -> 10K
- R37, R38, R39, R40, R41: footprint Resistor_SMD:R_0603_1608Metric -> Resistor_SMD:R_0402_1005Metric
Routing:
- net GND: track 180.7 -> 179.8 mm, vias 68 -> 66
Other:
- board text added: "BETA TEST EDITION"
- board text added: "Version 5.3.0"
- board text removed: "Version 5.3.0 Beta test edition"
