File: 2_prototype_mk5/hardware/HDD Synth Prototype MK5.kicad_sch (KiCad schematic)
At the start: 14 parts, among them U1 Optocoupler_DC_PhotoNPN_AKEC

Commit message: MKV revision 1
Parts:
- removed H4, H5, H6, H7: MountingHole, MountingHole:MountingHole_3.2mm_M3, symbol Mechanical:MountingHole
- H1, H2, H3: LCSC Part Number (none) -> C124375; LCSC_Part_Number C124375 -> (none)
- H10, H11, H8, H9: now not fitted
- R1, R2: LCSC Part Number (none) -> C23138; LCSC_Part_Number C23138 -> (none)
- U1: LCSC Part Number (none) -> C2916312; LCSC_Part_Number C2916312 -> (none)
Other:
- sheet Power ports: added none; removed 5V_POWER
- sheet RGB LED ports: added RGB_LED_BLUE, RGB_LED_GREEN, RGB_LED_RED; removed RGB_DATA
- sheet RP2350 ports: added GPIO04_RGB_LED_RED, GPIO05_RGB_LED_GREEN, GPIO06_RGB_LED_BLUE; removed GPIO07_LED_DATA
- note removed: "Speaker mounts (Small) Dimensions: 40x40x20mm"

Commit message: MKV revision 1 enhancements
- RGB LED support
- 3D printable 3.5/2.5" drive bay mounts
Parts:
- U1: LCSC Part Number C2916312 -> C42381015
Changed lines of the file:
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@@
 			)
 		)
-		(property "LCSC Part Number" "C2916312"
+		(property "LCSC Part Number" "C42381015"
 			(at 38.1 173.99 0)
 			(hide yes)

Commit message: Add buck boost to 5V and reset line stability
Other:
- sheet Power ports: added PG_STATUS, VCAP_DETECT; removed none
- sheet RP2350 ports: added GPIO27_ADC1_VCAP_DETECT; removed none
Changed lines of the file:
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@@
 	(wire
 		(pts
+			(xy 166.37 109.22) (xy 182.88 109.22)
+		)
+		(stroke
+			(width 0)
+			(type default)
+		)
+	)
+	(wire
+		(pts
 			(xy 166.37 82.55) (xy 181.61 82.55)
 		)
@@
 	(sheet
 		(at 182.88 104.14)
-		(size 24.13 7.62)
+		(size 24.13 8.89)
 		(exclude_from_sim no)
 		(in_bom yes)
@@
 		)
 		(property "Sheetfile" "power.kicad_sch"
-			(at 182.88 112.3446 0)
+			(at 182.88 113.6146 0)
 			(show_name no)
 			(do_not_autoplace no)
@@
 			)
 		)
+		(pin "PG_STATUS" output
+			(at 182.88 111.76 180)
+			(effects
+				(font
+					(size 1.27 1.27)
+				)
+				(justify left)
+			)
+		)
+		(pin "VCAP_DETECT" output
+			(at 182.88 109.22 180)
+			(effects
+				(font
+					(size 1.27 1.27)
+				)
+				(justify left)
+			)
+		)
 		(instances
 			(project "HDD Synth Prototype MK5"
@@
 			)
 		)
+		(pin "GPIO27_ADC1_VCAP_DETECT" bidirectional
+			(at 166.37 109.22 0)
+			(effects
+				(font
+					(size 1.27 1.27)
+				)
+				(justify right)
+			)
+		)

Commit message: Cost reductions for JCLPCB
Parts:
- H1, H2, H3: now not fitted; now left out of the parts list
Other:
- sheet Power ports: added none; removed PG_STATUS
- sheet RP2350 ports: added GPIO24_OLED_SDA, GPIO25_OLED_SCL; removed GPIO23_OLED_SDA, GPIO24_OLED_SCL
Changed lines of the file:
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@@
 		(body_style 1)
 		(exclude_from_sim no)
-		(in_bom yes)
+		(in_bom no)
 		(on_board yes)
 		(in_pos_files yes)
-		(dnp no)
+		(dnp yes)
 		(property "Reference" "H2"
 			(at 29.21 137.1599 0)
@@
 		(body_style 1)
 		(exclude_from_sim no)
-		(in_bom yes)
+		(in_bom no)
 		(on_board yes)
 		(in_pos_files yes)
-		(dnp no)
+		(dnp yes)
 		(fields_autoplaced yes)
 		(property "Reference" "H3"
@@
 		(body_style 1)
 		(exclude_from_sim no)
-		(in_bom yes)
+		(in_bom no)
 		(on_board yes)
 		(in_pos_files yes)
-		(dnp no)
+		(dnp yes)
 		(property "Reference" "H1"
 			(at 27.94 102.8699 0)
@@
 			)
 		)
-		(pin "PG_STATUS" output
-			(at 182.88 111.76 180)
-			(effects
-				(font
-					(size 1.27 1.27)
-				)
-				(justify left)
-			)
-		)
 		(pin "VCAP_DETECT" output
 			(at 182.88 109.22 180)
@@
 			)
 		)
-		(pin "GPIO23_OLED_SDA" bidirectional
-			(at 123.19 85.09 180)
-			(effects
-				(font
-					(size 1.27 1.27)
-				)
-				(justify left)
-			)
-		)
-		(pin "GPIO24_OLED_SCL" bidirectional
-			(at 123.19 87.63 180)
-			(effects
-				(font
-					(size 1.27 1.27)
-				)
-				(justify left)
-			)
-		)
 		(pin "GPIO04_RGB_LED_RED" bidirectional
 			(at 123.19 114.3 180)
@@
 			)
 		)
+		(pin "GPIO24_OLED_SDA" bidirectional
+			(at 123.19 85.09 180)
+			(effects
+				(font
+					(size 1.27 1.27)
+				)
+				(justify left)
+			)
+		)
+		(pin "GPIO25_OLED_SCL" bidirectional
+			(at 123.19 87.63 180)
+			(effects
+				(font
+					(size 1.27 1.27)
+				)
+				(justify left)
+			)
+		)
