File: 2_prototype_mk5/hardware/HDD Synth Prototype MK5.kicad_sch (KiCad schematic)
At the start: 10 parts, among them U1 Optocoupler_DC_PhotoNPN_AKEC

Commit message: MK5 revision 2 hardware updates and ISA adapter revisions
Ignore VSCode local-history artifacts going forward.

Co-Authored-By: Claude Sonnet 5 <noreply@anthropic.com>
Parts:
- H1, H2, H3: now fitted; now in the parts list
Changed lines of the file:
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@@
 		(body_style 1)
 		(exclude_from_sim no)
-		(in_bom no)
+		(in_bom yes)
 		(on_board yes)
 		(in_pos_files yes)
-		(dnp yes)
+		(dnp no)
 		(property "Reference" "H2"
 			(at 29.21 137.1599 0)
@@
 		(body_style 1)
 		(exclude_from_sim no)
-		(in_bom no)
+		(in_bom yes)
 		(on_board yes)
 		(in_pos_files yes)
-		(dnp yes)
+		(dnp no)
 		(fields_autoplaced yes)
 		(property "Reference" "H3"
@@
 		(body_style 1)
 		(exclude_from_sim no)
-		(in_bom no)
+		(in_bom yes)
 		(on_board yes)
 		(in_pos_files yes)
-		(dnp yes)
+		(dnp no)
 		(property "Reference" "H1"
 			(at 27.94 102.8699 0)
