File: 2_prototype_mk5/hardware/HDD Synth Prototype MK5.kicad_sch (KiCad schematic)
At the start: 10 parts, among them U1 Optocoupler_DC_PhotoNPN_AKEC

Commit message: Tweaks
Other:
- sheet Power ports: added PWR_FAULT_N, VSUP_SENSE; removed VCAP_DETECT, VCC_DETECT_POWER
- sheet RP2350 ports: added GPIO27_ADC1_PWR_FAULT_N, GPIO28_ADC2_VSUP_SENSE; removed GPIO27_ADC1_VCAP_DETECT, GPIO28_ADC2_VCC_DETECT
Changed lines of the file:
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@@
 			)
 		)
-		(pin "VCC_DETECT_POWER" output
+		(pin "PWR_FAULT_N" output
 			(at 182.88 106.68 180)
 			(effects
@@
 			)
 		)
-		(pin "VCAP_DETECT" output
+		(pin "VSUP_SENSE" output
 			(at 182.88 109.22 180)
 			(effects
@@
 			)
 		)
-		(pin "GPIO28_ADC2_VCC_DETECT" bidirectional
-			(at 166.37 106.68 0)
-			(effects
-				(font
-					(size 1.27 1.27)
-				)
-				(justify right)
-			)
-		)
 		(pin "GPIO04_RGB_LED_RED" bidirectional
 			(at 123.19 114.3 180)
@@
 			)
 		)
-		(pin "GPIO27_ADC1_VCAP_DETECT" bidirectional
-			(at 166.37 109.22 0)
-			(effects
-				(font
-					(size 1.27 1.27)
-				)
-				(justify right)
-			)
-		)
 		(pin "GPIO24_OLED_SDA" bidirectional
 			(at 123.19 85.09 180)
@@
 			)
 		)
+		(pin "GPIO27_ADC1_PWR_FAULT_N" bidirectional
+			(at 166.37 106.68 0)
+			(effects
+				(font
+					(size 1.27 1.27)
+				)
+				(justify right)
+			)
+		)
+		(pin "GPIO28_ADC2_VSUP_SENSE" bidirectional
+			(at 166.37 109.22 0)
+			(effects
+				(font
+					(size 1.27 1.27)
+				)
+				(justify right)
+			)
+		)

Commit message: Tweaks
Other:
- sheet RP2350 ports: added GPIO27_ADC1_VSUP_SENSE, GPIO28_ADC2_PWR_FAULT_N; removed GPIO27_ADC1_PWR_FAULT_N, GPIO28_ADC2_VSUP_SENSE
Changed lines of the file:
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@@
 			)
 		)
-		(pin "GPIO27_ADC1_PWR_FAULT_N" bidirectional
+		(pin "GPIO28_ADC2_PWR_FAULT_N" bidirectional
 			(at 166.37 106.68 0)
 			(effects
@@
 			)
 		)
-		(pin "GPIO28_ADC2_VSUP_SENSE" bidirectional
+		(pin "GPIO27_ADC1_VSUP_SENSE" bidirectional
 			(at 166.37 109.22 0)
 			(effects
