File: 2_prototype_mk5/hardware/RP2350_60QFN_minimal.kicad_sch (KiCad schematic)
At the start: 39 parts, among them J2 Conn_01x03, J4 USB_C_Receptacle_USB2.0_16P, SW1 SW_Push, SW2 SW_Push, U3 W25Q128JVS, U4 NCP1117-3.3_SOT223, U5 RP2350_60QFN, Y1 ABM8-272-T3

Commit message: Successful MKV software test (after minor modification)
Parts:
- removed SW1, SW2: SW_Push, Button_Switch_SMD:SW_Push_1P1T_NO_Vertical_Wuerth_434133025816, symbol Switch:SW_Push
- added S1, S2: TS-1187A-B-A-B, Custom:SW_TS-1187A-B-A-B, symbol Project symbols:TS-1187A-B-A-B
- J4: footprint Connector_USB:USB_C_Receptacle_Amphenol_12401610E4-2A -> Connector_USB:USB_C_Receptacle_HRO_TYPE-C-31-M-12; LCSC_Part_Number C5119948 -> C165948
- R15, R16: LCSC_Part_Number (none) -> C138021
Connections:
- net GND: now also S2.A, S2.B
- net RUN: now also S1.C, S1.D
- net ~{USB_BOOT}: now also S2.C, S2.D
- net at R12.1: now also S1.A, S1.B
Other:
- moved on the sheet: R12

Commit message: MKV revision 1
Parts:
- C10, C14, C17, C18, C19, C20, C21, C22, C23, C24: LCSC Part Number (none) -> C1525; LCSC_Part_Number C1525 -> (none)
- C11, C25, C9: LCSC Part Number (none) -> C15850; LCSC_Part_Number C15850 -> (none)
- C12, C13, C15, C16: LCSC Part Number (none) -> C23733; LCSC_Part_Number C23733 -> (none)
- C7, C8: LCSC Part Number (none) -> C1548; LCSC_Part_Number C1548 -> (none)
- J2: LCSC Part Number (none) -> C49257; LCSC_Part_Number C49257 -> (none)
- J4: LCSC Part Number (none) -> C165948; LCSC_Part_Number C165948 -> (none)
- L1: LCSC Part Number (none) -> C42411119; LCSC_Part_Number C42411119 -> (none)
- R10, R12, R14: LCSC Part Number (none) -> C11702; LCSC_Part_Number C11702 -> (none)
- R11, R8: LCSC Part Number (none) -> C25905; LCSC_Part_Number C25905 -> (none)
- R13: LCSC Part Number (none) -> C25105; LCSC_Part_Number C25105 -> (none)
- R15, R16: LCSC Part Number (none) -> C138021; LCSC_Part_Number C138021 -> (none)
- R6, R9: LCSC_Part_Number C25105 -> (none); now not fitted; now left out of the parts list
- R7: LCSC Part Number (none) -> C17168; LCSC_Part_Number C17168 -> (none)
- S1, S2: LCSC Part Number (none) -> C318884; LCSC_Part_Number C318884 -> (none)
- U3: value W25Q128JVS -> W25Q32JVSSIQ; LCSC Part Number (none) -> C179173; LCSC_Part_Number C83140 -> (none)
- U4: LCSC Part Number (none) -> C26537; LCSC_Part_Number C26537 -> (none)
- U5: LCSC Part Number (none) -> C42411118; LCSC_Part_Number C42411118 -> (none)
- Y1: LCSC Part Number (none) -> C20625731; LCSC_Part_Number C20625731 -> (none)
Connections:
- net GPIO07_LED_DATA renamed LED_DATA
- net GPIO4 renamed GPIO04_RGB_LED_RED
- net GPIO5 renamed GPIO05_RGB_LED_GREEN
- net GPIO6 renamed GPIO06_RGB_LED_BLUE
- no-connect marks 14 -> 12

Commit message: Add buck boost to 5V and reset line stability
Connections:
- net GPIO27_ADC1 renamed GPIO27_ADC1_VCAP_DETECT
- no-connect marks 12 -> 11
Changed lines of the file:
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@@
-	)
-	(no_connect
-		(at 306.07 176.53)
 	)
 	(no_connect
@@
 		)
 	)
-	(label "GPIO27_ADC1"
+	(label "VCAP_DETECT"
 		(at 306.07 176.53 180)
 		(effects
@@
 		(effects
 			(font
+				(size 1.27 1.27)
+			)
+			(justify left)
+		)
+	)
+	(hierarchical_label "GPIO27_ADC1_VCAP_DETECT"
+		(shape bidirectional)
+		(at 306.07 176.53 0)
+		(effects
+			(font

Commit message: Cost reductions for JCLPCB
Parts:
- J2, U3: now not fitted; now left out of the parts list
- R10, R12, R14: value 1k -> 1K
- R15, R16: LCSC Part Number C138021 -> C25100
- U5: LCSC Part Number C42411118 -> C41378174
Connections:
- net GPIO23_OLED_SDA renamed GPIO23
- net GPIO24_OLED_SCL renamed GPIO24_OLED_SDA
- net GPIO25 renamed GPIO25_OLED_SCL
Changed lines of the file:
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@@
 	)
 	(no_connect
+		(at 306.07 163.83)
+	)
+	(no_connect
 		(at 306.07 113.03)
 	)
@@
 	)
 	(no_connect
-		(at 306.07 168.91)
-	)
-	(no_connect
 		(at 306.07 146.05)
 	)
@@
 	(wire
 		(pts
-			(xy 290.83 166.37) (xy 306.07 166.37)
+			(xy 34.29 157.48) (xy 46.99 157.48)
 		)
 		(stroke
@@
 	(wire
 		(pts
-			(xy 34.29 157.48) (xy 46.99 157.48)
+			(xy 290.83 166.37) (xy 306.07 166.37)
 		)
 		(stroke
@@
 	(wire
 		(pts
-			(xy 290.83 163.83) (xy 306.07 163.83)
-		)
-		(stroke
-			(width 0)
-			(type default)
-		)
-	)
-	(wire
-		(pts
 			(xy 215.9 63.5) (xy 215.9 64.77)
 		)
@@
 	(wire
 		(pts
+			(xy 290.83 163.83) (xy 306.07 163.83)
+		)
+		(stroke
+			(width 0)
+			(type default)
+		)
+	)
+	(wire
+		(pts
 			(xy 175.26 158.75) (xy 180.34 158.75)
 		)
@@
 		)
 	)
-	(label "GPIO25"
+	(label "OLED_SCL"
 		(at 306.07 168.91 180)
 		(effects
@@
 		)
 	)
-	(label "OLED_SCL"
+	(label "OLED_SDA"
 		(at 306.07 166.37 180)
 		(effects
@@
 		)
 	)
-	(label "OLED_SDA"
+	(label "GPIO23"
 		(at 306.07 163.83 180)
 		(effects
@@
 		)
 	)
-	(hierarchical_label "GPIO24_OLED_SCL"
+	(hierarchical_label "GPIO25_OLED_SCL"
 		(shape bidirectional)
-		(at 306.07 166.37 0)
+		(at 306.07 168.91 0)
 		(effects
 			(font
@@
 		)
 	)
-	(hierarchical_label "GPIO23_OLED_SDA"
+	(hierarchical_label "GPIO24_OLED_SDA"
 		(shape bidirectional)
-		(at 306.07 163.83 0)
+		(at 306.07 166.37 0)
 		(effects
 			(font
@@
 		(body_style 1)
 		(exclude_from_sim no)
-		(in_bom yes)
+		(in_bom no)
 		(on_board yes)
 		(in_pos_files yes)
-		(dnp no)
+		(dnp yes)
 		(property "Reference" "U3"
 			(at 67.31 45.72 0)
@@
 			)
 		)
-		(property "LCSC Part Number" "C138021"
+		(property "LCSC Part Number" "C25100"
 			(at 306.07 88.9 90)
 			(hide yes)
@@
 			)
 		)
-		(property "LCSC Part Number" "C138021"
+		(property "LCSC Part Number" "C25100"
 			(at 306.07 97.79 90)
 			(hide yes)
@@
 			)
 		)
-		(property "Value" "1k"
+		(property "Value" "1K"
 			(at 171.45 155.8036 90)
 			(show_name no)
@@
 			)
 		)
-		(property "LCSC Part Number" "C42411118"
+		(property "LCSC Part Number" "C41378174"
 			(at 259.08 138.43 0)
 			(hide yes)
@@
 			)
 		)
-		(property "Value" "1k"
+		(property "Value" "1K"
 			(at 205.105 113.8936 90)
 			(show_name no)
@@
 		(body_style 1)
 		(exclude_from_sim no)
-		(in_bom yes)
+		(in_bom no)
 		(on_board yes)
 		(in_pos_files yes)
-		(dnp no)
+		(dnp yes)
 		(fields_autoplaced yes)
 		(property "Reference" "J2"
@@
 			)
 		)
-		(property "Value" "1k"
+		(property "Value" "1K"
 			(at 63.5 106.2736 90)
 			(show_name no)
