File: 2_prototype_mk5/hardware/RP2350_60QFN_minimal.kicad_sch (KiCad schematic)
At the start: 39 parts, among them J2 Conn_01x03, J4 USB_C_Receptacle_USB2.0_16P, U3 W25Q32JVSSIQ, U4 NCP1117-3.3_SOT223, U5 RP2350_60QFN, Y1 ABM8-272-T3

Commit message: MK5 revision 2 hardware updates and ISA adapter revisions
Ignore VSCode local-history artifacts going forward.

Co-Authored-By: Claude Sonnet 5 <noreply@anthropic.com>
Parts:
- J2: now fitted; now in the parts list
Changed lines of the file:
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@@
 		(body_style 1)
 		(exclude_from_sim no)
-		(in_bom no)
+		(in_bom yes)
 		(on_board yes)
 		(in_pos_files yes)
-		(dnp yes)
+		(dnp no)
 		(fields_autoplaced yes)
 		(property "Reference" "J2"
