File: 2_prototype_mk5/hardware/RP2350_60QFN_minimal.kicad_sch (KiCad schematic)
At the start: 39 parts, among them J2 Conn_01x03, J4 USB_C_Receptacle_USB2.0_16P, U3 W25Q32JVSSIQ, U4 NCP1117-3.3_SOT223, U5 RP2350_60QFN, Y1 ABM8-272-T3

Commit message: eFuse and regular
Connections:
- net VBUS renamed VIN_RAW
Changed lines of the file:
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@@
 			)
 		)
-		(property "Value" "VBUS"
+		(property "Value" "VIN_RAW"
 			(at 51.181 198.8058 0)
 			(show_name no)

Commit message: Tweaks
Parts:
- removed C11, C9: 10uF, Capacitor_SMD:C_0805_2012Metric, symbol Device:C
- removed U4: NCP1117-3.3_SOT223, Package_TO_SOT_SMD:SOT-223-3_TabPin2, symbol Regulator_Linear:NCP1117-3.3_SOT223
Connections:
- net GPIO27_ADC1_VCAP_DETECT renamed GPIO27_ADC1_PWR_FAULT_N
- net GPIO28_ADC2_VCC_DETECT renamed GPIO28_ADC2_VSUP_SENSE
