File: 2_prototype_mk5/hardware/RP2350_60QFN_minimal.kicad_sch (KiCad schematic)
At the start: 36 parts, among them J2 Conn_01x03, J4 USB_C_Receptacle_USB2.0_16P, U3 W25Q32JVSSIQ, U5 RP2350_60QFN, Y1 ABM8-272-T3

Commit message: Tweaks
Connections:
- net GPIO27_ADC1_PWR_FAULT_N renamed GPIO27_ADC1_VSUP_SENSE
- net GPIO28_ADC2_VSUP_SENSE renamed GPIO28_ADC2_PWR_FAULT_N
Changed lines of the file:
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@@
 		)
 	)
-	(label "VCAP_DETECT"
+	(label "VSUP_SENSE"
 		(at 306.07 176.53 180)
 		(effects
@@
 		)
 	)
-	(hierarchical_label "GPIO27_ADC1_PWR_FAULT_N"
+	(hierarchical_label "GPIO27_ADC1_VSUP_SENSE"
 		(shape bidirectional)
 		(at 306.07 176.53 0)
@@
 		)
 	)
-	(hierarchical_label "GPIO28_ADC2_VSUP_SENSE"
+	(hierarchical_label "GPIO28_ADC2_PWR_FAULT_N"
 		(shape bidirectional)
 		(at 306.07 179.07 0)
