File: 2_prototype_mk5/hardware/RP2350_60QFN_minimal.kicad_sch (KiCad schematic)
At the start: 36 parts, among them J2 Conn_01x03, J4 USB_C_Receptacle_USB2.0_16P, U3 W25Q32JVSSIQ, U5 RP2350_60QFN, Y1 ABM8-272-T3

Commit message: 5.3.0 sent to JCLPCB
Parts:
- Y1: LCSC Part Number C20625731 -> C20617575
Changed lines of the file:
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@@
 			)
 		)
-		(property "LCSC Part Number" "C20625731"
+		(property "LCSC Part Number" "C20617575"
 			(at 45.72 104.14 90)
 			(hide yes)
