File: 2_prototype_mk5/hardware/power.kicad_sch (KiCad schematic)
At the start: 21 parts, among them U6 TPS63020DSJR

Commit message: eFuse and regular
Parts:
- removed D1, D2: SS14, Diode_SMD:D_SMA, symbol Device:D_Schottky
- removed R3, R4: 10K, Resistor_SMD:R_0603_1608Metric, symbol Device:R
- removed R5: 22R, Resistor_SMD:R_2512_6332Metric, symbol Device:R
- added C34: 4.7nF, Capacitor_SMD:C_0402_1005Metric, symbol Device:C
- added C35: 1uF, Capacitor_SMD:C_0402_1005Metric, symbol Device:C
- added C36, C37: 10uF, Capacitor_SMD:C_0805_2012Metric, symbol Device:C
- added L2: L, symbol Device:L
- added R32: 360K, Resistor_SMD:R_0402_1005Metric, symbol Device:R
- added R33: 33K, Resistor_SMD:R_0402_1005Metric, symbol Device:R
- added R34: 120K, Resistor_SMD:R_0402_1005Metric, symbol Device:R
- added R35: 100K, Resistor_SMD:R_0402_1005Metric, symbol Device:R
- added R36: 110K, Resistor_SMD:R_0402_1005Metric, symbol Device:R
- added R37, R38, R39: 75K, Resistor_SMD:R_0603_1608Metric, symbol Device:R
- added R40, R41: 100K, Resistor_SMD:R_0603_1608Metric, symbol Device:R
- added U8: TPS25921ADR, easyeda2kicad:SOIC-8_L5.0-W4.0-P1.27-LS6.0-BL, symbol easyeda2kicad:TPS25921ADR
- added U9: TPS61094DSSR, easyeda2kicad:WSON-12_L3.0-W2.0-P0.5-BL-EP, symbol easyeda2kicad:TPS61094DSSR
- R31: value 100K -> 24K; LCSC Part Number C25741 -> (none)
- Super_Cap1: value 1F -> 1.5F
Connections:
- net +5V: now also C35.2, R32.1, U8.4 (IN)
- net GND: now also C34.2, C35.1, C36.1, C37.2, R34.2, R36.2, R37.2, R38.1, R39.1, U8.1 (GND), U9.13 (EP), U9.7 (PGND), U9.8 (AGND)
- net at Super_Cap1.1: now also C36.2, L2.2, U9.6 (SUP)
- net POWER_5V_SUP renamed +3.3V
- net VCAP_RAW renamed VSYS
- net VSYS: now also R40.2, R41.2, U9.10 (VOUT), U9.9 (VOUT); no longer R24.2
- new net: L2.1, U9.5 (SW)
- new net: R33.1, R34.1, U8.8 (OVP)
- new net: R41.1, U9.3 (EN)
- new net: R32.2, R33.2, U8.3 (ENUV)
- new net: C34.1, U8.2 (SS)
- new net: R37.1, U9.1 (OSEL)
- new net: R35.1, U8.6 (#FLT)
- new net: R39.2, U9.12 (VCHG)
- new net: R36.1, U8.7 (ILIM)
- new net: R40.1, U9.2 (MODE)
- new net: R38.2, U9.11 (ICHG)
- new net +3V3: R35.2
- new net VIN_PROT: C37.1, R24.2, U8.5 (OUT), U9.4 (VIN)
Other:
- note added: "- 4.5 V to 18 V operating range - Programmable 0.4 A to 1.6 A current limit - Integrated 90ohm power MOSFET - Overcurrent & fast short-circuit protection - Overvoltage protection (OVP) & UVLO - Soft-start inrush current control"
- note added: "3.3v output"
- note added: "Buck boost to 3.3v output"
- note added: "Electro cap"
- note added: "It's an open-drain output that goes low on three conditions: undervoltage, overvoltage, and thermal shutdown. A nuisance fast-trip doesn't trigger it. Connect to GPIO to detect - So external power off"
- note added: "Not needed anymore (Check)"
- note added: "Potential use in future revision, but not used currently due to complexity of routing and marginal benefits"
- note added: "USB C power"
- note added: "VCHG: 4.15v termination ICHG: 250mA charge"
- note added: "What current limit is set?"
- note added: "eFuse"
- note removed: "Buck boost 5v"
- note removed: "Changed from original R22 180K / R21 1.6M in spec sheet to LCSC basic parts to save money, but keep same voltage divider"
- note removed: "Ensure when running on super cap that voltage is always regulated to 5v"
- note removed: "External voltage detection"
- note removed: "Halves the voltage (5v external to 2.5v)"
- note removed: "Planned for revision 2, but not used due to complexity of routing and marginal benefits"
- moved on the sheet: C27, C28, C29, C30, C31, C32, C33, H14, L3, R22, R24, R25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

Commit message: Tweaks
Parts:
- added C38: 100uF, Capacitor_SMD:CP_Elec_6.3x7.7, symbol Device:C_Polarized
Connections:
- net +3V3: now also C29.1, R31.1, U6.4 (VOUT), U6.5 (VOUT)
- net GND: now also C38.2
- net VIN_PROT: now also C38.1; no longer R24.2
- net VSYS: now also C31.1, C32.1
- net at C36.2, L2.2, Super_Cap1.1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: now also R24.2
- removed net +3.3V: C29.1, C31.1, C32.1, R31.1, U6.4 (VOUT), U6.5 (VOUT)
Other:
- note removed: "Electro cap"
- moved on the sheet: C27, C28, C29, C30, C33, C37, R24, R25

Commit message: Tweaks
Parts:
- L2: value L -> 2.2 µH; footprint (none) -> easyeda2kicad:IND-SMD_L4.0-W4.0_FNR40XXS
Connections:
- net +3V3: now also C32.2
- net GND: now also C32.1; no longer C32.2
- net VSYS: no longer C32.1
Other:
- moved on the sheet: C33, C36, C37, C38, L2, R24, R25, R37, R38, R39, R40, R41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

Commit message: Tweaks
Connections:
- net PWR_FAULT_N: now reaches R35.1, U8.6 (#FLT)
- net VCAP_DETECT renamed VSUP_SENSE
Other:
- note added: "Open-drain output that goes low on three conditions: - undervoltage - overvoltage - thermal shutdown"
- note removed: "It's an open-drain output that goes low on three conditions: undervoltage, overvoltage, and thermal shutdown. A nuisance fast-trip doesn't trigger it. Connect to GPIO to detect - So external power off"
- note removed: "Not needed anymore (Check)"
Changed lines of the file:
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@@
 		)
 	)
-	(text "It's an open-drain output that goes low on three conditions: \nundervoltage, overvoltage, and thermal shutdown. \nA nuisance fast-trip doesn't trigger it. Connect to GPIO to detect\n- So external power off"
+	(text "Open-drain output that goes \nlow on three conditions: \n- undervoltage\n- overvoltage\n- thermal shutdown"
 		(exclude_from_sim no)
-		(at 111.506 20.32 0)
+		(at 160.02 33.02 0)
 		(effects
 			(font
@@
 				(thickness 0.254)
 				(bold yes)
-				(color 255 0 13 1)
-			)
-			(justify left)
-		)
-	)
-	(text "Not needed anymore (Check)"
-		(exclude_from_sim no)
-		(at 236.22 149.606 0)
-		(effects
-			(font
-				(size 1.27 1.27)
-				(thickness 0.254)
-				(bold yes)
-				(color 255 0 13 1)
+				(color 0 0 255 1)
 			)
 			(justify left)
@@
 	(wire
 		(pts
-			(xy 139.7 27.94) (xy 139.7 60.96)
+			(xy 139.7 29.21) (xy 139.7 60.96)
 		)
 		(stroke
@@
 		(pts
 			(xy 71.12 144.78) (xy 74.93 144.78)
+		)
+		(stroke
+			(width 0)
+			(type default)
+		)
+	)
+	(wire
+		(pts
+			(xy 139.7 29.21) (xy 142.24 29.21)
 		)
 		(stroke
@@
 		)
 	)
-	(label "VCAP_DETECT"
+	(label "VSUP_SENSE"
 		(at 236.22 144.78 0)
 		(effects
@@
 		)
 	)
-	(hierarchical_label "VCAP_DETECT"
+	(hierarchical_label "PWR_FAULT_N"
+		(shape output)
+		(at 142.24 29.21 0)
+		(effects
+			(font
+				(size 1.27 1.27)
+			)
+			(justify left)
+		)
+	)
+	(hierarchical_label "VSUP_SENSE"
 		(shape output)
 		(at 251.46 144.78 0)

Commit message: Tweaks
Parts:
- added D1: SMAJ5.0A, Diode_SMD:D_SMA, symbol Device:D_Zener
Connections:
- net +5V: now also D1.2 (A); no longer C35.2, R32.1, U8.4 (IN)
- new net: C35.2, D1.1 (K), R32.1, U8.4 (IN)

Commit message: Tweaks
Parts:
- added C39: 22uF, Capacitor_SMD:C_0805_2012Metric, symbol Device:C
Connections:
- net +5V: now also C35.2, D1.1 (K), R32.1, U8.4 (IN); no longer D1.2 (A)
- net GND: now also D1.2 (A), C39.2
- net VSYS: now also C39.1
Other:
- moved on the sheet: D1

Commit message: Tweaks
Parts:
- R32: value 360K -> 330K
- R33: value 33K -> 47K
Other:
- note added: "- Configured for 5 V input - Overvoltage cutoff at 5.76 V, undervoltage at 4.14 V - Programmable current limit set to 1.16 A (1.92 A fast short-circuit trip) - Integrated 87 mΩ power MOSFET - 4.9 ms soft-start ramp limits inrush to ~110 mA - Open-drain fault flag to GP28 for hardware power-fail detection"
- note removed: "- 4.5 V to 18 V operating range - Programmable 0.4 A to 1.6 A current limit - Integrated 90ohm power MOSFET - Overcurrent & fast short-circuit protection - Overvoltage protection (OVP) & UVLO - Soft-start inrush current control"
- note removed: "What current limit is set?"
Changed lines of the file:
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@@
 	)
 	(rectangle
-		(start 49.53 26.67)
+		(start 49.53 20.32)
 		(end 158.75 87.63)
 		(stroke
@@
 		)
 	)
-	(text "- 4.5 V to 18 V operating range \n- Programmable 0.4 A to 1.6 A current limit\n- Integrated 90ohm  power MOSFET\n- Overcurrent & fast short-circuit protection\n- Overvoltage protection (OVP) & UVLO\n- Soft-start inrush current control"
+	(text "- Configured for 5 V input\n- Overvoltage cutoff at 5.76 V, \n  undervoltage at 4.14 V\n- Programmable current limit set to 1.16 A \n  (1.92 A fast short-circuit trip)\n- Integrated 87 mΩ power MOSFET\n- 4.9 ms soft-start ramp limits inrush to ~110 mA\n- Open-drain fault flag to GP28 for \n  hardware power-fail detection"
 		(exclude_from_sim no)
-		(at 51.308 36.576 0)
+		(at 51.562 33.528 0)
 		(effects
 			(font
@@
 	(text "eFuse"
 		(exclude_from_sim no)
-		(at 54.356 28.956 0)
+		(at 54.356 23.114 0)
 		(effects
 			(font
@@
 		)
 	)
-	(text "What current limit is set?"
-		(exclude_from_sim no)
-		(at 72.644 24.384 0)
-		(effects
-			(font
-				(size 1.27 1.27)
-				(thickness 0.254)
-				(bold yes)
-				(color 255 0 0 1)
-			)
-		)
-	)
 	(text "Spin down power reserve"
 		(exclude_from_sim no)
@@
 			)
 		)
-		(property "Value" "33K"
+		(property "Value" "47K"
 			(at 116.84 52.07 90)
 			(show_name no)
@@
 			)
 		)
-		(property "Value" "360K"
+		(property "Value" "330K"
 			(at 57.15 57.15 90)
 			(show_name no)
