File: 2_prototype_mk5/hardware/power.kicad_sch (KiCad schematic)
At the start: 36 parts, among them U6 TPS63020DSJR, U8 TPS25921ADR, U9 TPS61094DSSR

Commit message: Schematics and layout complete for 5.2.0
Co-Authored-By: Claude Sonnet 5 <noreply@anthropic.com>
Parts:
- Super_Cap1: footprint Capacitor_THT:CP_Radial_D14.0mm_P5.00mm -> Custom:SuperCap_Eaton_PHV_9.0x17.3mm_P11.80mm
Changed lines of the file:
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@@
 			)
 		)
-		(property "Footprint" "Capacitor_THT:CP_Radial_D14.0mm_P5.00mm"
+		(property "Footprint" "Custom:SuperCap_Eaton_PHV_9.0x17.3mm_P11.80mm"
 			(at 215.9 116.84 0)
 			(hide yes)
