File: 2_prototype_mk5/hardware/power.kicad_sch (KiCad schematic)
At the start: 36 parts, among them U6 TPS63020DSJR, U8 TPS25921ADR, U9 TPS61094DSSR

Commit message: Tweaks
Parts:
- R35: value 100K -> 10K
Changed lines of the file:
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@@
 			)
 		)
-		(property "Value" "100K"
+		(property "Value" "10K"
 			(at 144.78 57.15 90)
 			(show_name no)

Commit message: 5.3.0 sent to JCLPCB
Parts:
- C38: LCSC Part Number (none) -> C134801
- L2: LCSC Part Number (none) -> C167804
- L3: LCSC Part C167802 -> (none); LCSC Part Number (none) -> C167802
- R31: value 24K -> 22K; LCSC Part Number (none) -> C25768
- R32: LCSC Part Number (none) -> C25778
- R33: LCSC Part Number (none) -> C25792
- R34: LCSC Part Number (none) -> C25750
- R35: LCSC Part Number (none) -> C25744
- R36: value 110K -> 120K; LCSC Part Number (none) -> C25750
- R37, R38, R39: footprint Resistor_SMD:R_0603_1608Metric -> Resistor_SMD:R_0402_1005Metric; LCSC Part Number (none) -> C25798
- R40, R41: footprint Resistor_SMD:R_0603_1608Metric -> Resistor_SMD:R_0402_1005Metric; LCSC Part Number (none) -> C25741
- U6: LCSC Part C15483 -> (none); LCSC Part Number (none) -> C15483
- U8: LCSC Part C189199 -> (none); LCSC Part Number (none) -> C189199
- U9: LCSC Part C3034939 -> (none); LCSC Part Number (none) -> C3034939
Changed lines of the file:
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@@
 			)
 		)
+		(property "LCSC Part Number" "C167804"
+			(at 199.39 109.22 0)
+			(hide yes)
+			(show_name no)
+			(do_not_autoplace no)
+			(effects
+				(font
+					(size 1.27 1.27)
+				)
+			)
+		)
 		(pin "2"
 		)
@@
 			)
 		)
-		(property "LCSC Part Number" ""
+		(property "LCSC Part Number" "C25750"
 			(at 116.84 38.1 90)
 			(hide yes)
@@
 			)
 		)
-		(property "Footprint" "Resistor_SMD:R_0603_1608Metric"
+		(property "Footprint" "Resistor_SMD:R_0402_1005Metric"
 			(at 200.66 98.552 90)
 			(hide yes)
@@
 			)
 		)
-		(property "LCSC Part Number" ""
+		(property "LCSC Part Number" "C25741"
 			(at 200.66 100.33 0)
 			(hide yes)
@@
 			)
 		)
-		(property "LCSC Part" "C167802"
+		(property "LCSC Part" ""
 			(at 102.87 190.5 0)
 			(hide yes)
@@
 			)
 		)
+		(property "LCSC Part Number" "C167802"
+			(at 102.87 172.72 0)
+			(hide yes)
+			(show_name no)
+			(do_not_autoplace no)
+			(effects
+				(font
+					(size 1.27 1.27)
+				)
+			)
+		)
 		(pin "2"
 		)
@@
 			)
 		)
-		(property "LCSC Part" "C15483"
+		(property "LCSC Part" ""
 			(at 102.87 180.34 0)
 			(hide yes)
@@
 			)
 		)
+		(property "LCSC Part Number" "C15483"
+			(at 102.87 149.86 0)
+			(hide yes)
+			(show_name no)
+			(do_not_autoplace no)
+			(effects
+				(font
+					(size 1.27 1.27)
+				)
+			)
+		)
 		(pin "6"
 		)
@@
 			)
 		)
-		(property "LCSC Part Number" ""
+		(property "LCSC Part Number" "C25792"
 			(at 116.84 55.88 90)
 			(hide yes)
@@
 			)
 		)
-		(property "Footprint" "Resistor_SMD:R_0603_1608Metric"
+		(property "Footprint" "Resistor_SMD:R_0402_1005Metric"
 			(at 214.63 93.472 90)
 			(hide yes)
@@
 			)
 		)
-		(property "LCSC Part Number" ""
+		(property "LCSC Part Number" "C25798"
 			(at 214.63 95.25 0)
 			(hide yes)
@@
 			)
 		)
-		(property "LCSC Part Number" ""
+		(property "LCSC Part Number" "C25744"
 			(at 144.78 60.96 90)
 			(hide yes)
@@
 			)
 		)
-		(property "Footprint" "Resistor_SMD:R_0603_1608Metric"
+		(property "Footprint" "Resistor_SMD:R_0402_1005Metric"
 			(at 248.92 93.472 90)
 			(hide yes)
@@
 			)
 		)
-		(property "LCSC Part Number" ""
+		(property "LCSC Part Number" "C25798"
 			(at 248.92 95.25 0)
 			(hide yes)
@@
 			)
 		)
-		(property "LCSC Part" "C189199"
+		(property "LCSC Part" ""
 			(at 96.52 81.28 0)
 			(hide yes)
@@
 			)
 		)
+		(property "LCSC Part Number" "C189199"
+			(at 96.52 59.69 0)
+			(hide yes)
+			(show_name no)
+			(do_not_autoplace no)
+			(effects
+				(font
+					(size 1.27 1.27)
+				)
+			)
+		)
 		(pin "7"
 		)
@@
 			)
 		)
-		(property "Footprint" "Resistor_SMD:R_0603_1608Metric"
+		(property "Footprint" "Resistor_SMD:R_0402_1005Metric"
 			(at 208.28 96.012 90)
 			(hide yes)
@@
 			)
 		)
-		(property "LCSC Part Number" ""
+		(property "LCSC Part Number" "C25741"
 			(at 208.28 97.79 0)
 			(hide yes)
@@
 			)
 		)
-		(property "Footprint" "Resistor_SMD:R_0603_1608Metric"
+		(property "Footprint" "Resistor_SMD:R_0402_1005Metric"
 			(at 256.54 96.012 90)
 			(hide yes)
@@
 			)
 		)
-		(property "LCSC Part Number" ""
+		(property "LCSC Part Number" "C25798"
 			(at 256.54 97.79 0)
 			(hide yes)
@@
 			)
 		)
-		(property "Value" "24K"
+		(property "Value" "22K"
 			(at 57.15 140.97 90)
 			(show_name no)
@@
 			)
 		)
-		(property "LCSC Part Number" ""
+		(property "LCSC Part Number" "C25768"
 			(at 57.15 144.78 90)
 			(hide yes)
@@
 			)
 		)
-		(property "LCSC Part" "C3034939"
+		(property "LCSC Part" ""
 			(at 231.14 125.73 0)
 			(hide yes)
@@
 			)
 		)
+		(property "LCSC Part Number" "C3034939"
+			(at 231.14 100.33 0)
+			(hide yes)
+			(show_name no)
+			(do_not_autoplace no)
+			(effects
+				(font
+					(size 1.27 1.27)
+				)
+			)
+		)
 		(pin "12"
 		)
@@
 			)
 		)
-		(property "LCSC Part Number" ""
+		(property "LCSC Part Number" "C25778"
 			(at 57.15 60.96 90)
 			(hide yes)
@@
 			)
 		)
+		(property "LCSC Part Number" "C134801"
+			(at 179.07 99.06 0)
+			(hide yes)
+			(show_name no)
+			(do_not_autoplace no)
+			(effects
+				(font
+					(size 1.27 1.27)
+				)
+			)
+		)
 		(pin "1"
 		)
@@
 			)
 		)
-		(property "Value" "110K"
+		(property "Value" "120K"
 			(at 128.27 54.61 90)
 			(show_name no)
@@
 			)
 		)
-		(property "LCSC Part Number" ""
+		(property "LCSC Part Number" "C25750"
 			(at 128.27 58.42 90)
 			(hide yes)
