File: 2_prototype_mk5/hardware/amplifier.kicad_sch (KiCad schematic)
At the start: 8 parts, among them U2 MAX98357A

Commit message: Successful MKV software test (after minor modification)
Parts:
- C2: LCSC_Part_Number C13585 -> C77093
Changed lines of the file:
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@@
 			)
 		)
-		(property "LCSC_Part_Number" "C13585"
+		(property "LCSC_Part_Number" "C77093"
 			(at 160.02 64.77 0)
 			(hide yes)

Commit message: MKV revision 1
Parts:
- C1: LCSC Part Number (none) -> C14663; LCSC_Part_Number C14663 -> (none)
- C2: LCSC Part Number (none) -> C14860; LCSC_Part_Number C77093 -> (none)
- C3, C4: LCSC Part Number (none) -> C1588; LCSC_Part_Number C1588 -> (none)
- FB1, FB2: LCSC Part Number (none) -> C85840; LCSC_Part_Number C85840 -> (none)
- H12: LCSC Part Number (none) -> C3819527; LCSC_Part_Number C3819527 -> (none)
- U2: LCSC Part Number (none) -> C910544; LCSC_Part_Number C910544 -> (none)
Changed lines of the file:
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@@
+	)
+	(junction
+		(at 149.86 77.47)
+		(diameter 0)
+		(color 0 0 0 0)
 	)
 	(junction
@@
 	(wire
 		(pts
-			(xy 149.86 60.96) (xy 149.86 92.71)
+			(xy 149.86 60.96) (xy 149.86 77.47)
 		)
 		(stroke
@@
 		(pts
 			(xy 121.92 110.49) (xy 137.16 110.49)
+		)
+		(stroke
+			(width 0)
+			(type default)
+		)
+	)
+	(wire
+		(pts
+			(xy 149.86 77.47) (xy 149.86 92.71)
 		)
 		(stroke
@@
 			)
 		)
-		(property "LCSC_Part_Number" "C1588"
-			(at 187.96 96.52 0)
-			(hide yes)
-			(show_name no)
-			(do_not_autoplace no)
-			(effects
-				(font
-					(size 1.27 1.27)
-				)
-			)
-		)
 		(property "Availability" ""
 			(at 187.96 96.52 0)
@@
 		)
 		(property "SnapEDA_Link" ""
+			(at 187.96 96.52 0)
+			(hide yes)
+			(show_name no)
+			(do_not_autoplace no)
+			(effects
+				(font
+					(size 1.27 1.27)
+				)
+			)
+		)
+		(property "LCSC Part Number" "C1588"
 			(at 187.96 96.52 0)
 			(hide yes)
@@
 				(path "/ed113b11-1722-4efb-9669-9e8c19f5c8fd/ceef9c1f-e4ce-45b2-b9fe-22340e8232b8"
 					(reference "C1")
+					(unit 1)
+				)
+			)
+		)
+	)
+	(symbol
+		(lib_id "power:PWR_FLAG")
+		(at 149.86 77.47 270)
+		(unit 1)
+		(body_style 1)
+		(exclude_from_sim no)
+		(in_bom yes)
+		(on_board yes)
+		(in_pos_files yes)
+		(dnp no)
+		(property "Reference" "#FLG05"
+			(at 151.765 77.47 0)
+			(hide yes)
+			(show_name no)
+			(do_not_autoplace no)
+			(effects
+				(font
+					(size 1.27 1.27)
+				)
+			)
+		)
+		(property "Value" "PWR_FLAG"
+			(at 154.94 80.01 0)
+			(show_name no)
+			(do_not_autoplace no)
+			(effects
+				(font
+					(size 1.27 1.27)
+				)
+			)
+		)
+		(property "Footprint" ""
+			(at 149.86 77.47 0)
+			(hide yes)
+			(show_name no)
+			(do_not_autoplace no)
+			(effects
+				(font
+					(size 1.27 1.27)
+				)
+			)
+		)
+		(property "Datasheet" ""
+			(at 149.86 77.47 0)
+			(hide yes)
+			(show_name no)
+			(do_not_autoplace no)
+			(effects
+				(font
+					(size 1.27 1.27)
+				)
+			)
+		)
+		(property "Description" "Special symbol for telling ERC where power comes from"
+			(at 149.86 77.47 0)
+			(hide yes)
+			(show_name no)
+			(do_not_autoplace no)
+			(effects
+				(font
+					(size 1.27 1.27)
+				)
+			)
+		)
+		(pin "1"
+		)
+		(instances
+			(project "HDD Synth Prototype MK5"
+				(path "/1a22431a-ba36-40a0-9a7e-c2a82ec69c53/2950dfc3-c685-4e23-94aa-d1af22619645"
+					(reference "#FLG05")
 					(unit 1)
 				)
@@
 			)
 		)
-		(property "LCSC_Part_Number" "C3819527"
-			(at 212.09 100.33 0)
-			(hide yes)
-			(show_name no)
-			(do_not_autoplace no)
-			(effects
-				(font
-					(size 1.27 1.27)
-				)
-			)
-		)
 		(property "Availability" ""
 			(at 212.09 100.33 0)
@@
 		)
 		(property "SnapEDA_Link" ""
+			(at 212.09 100.33 0)
+			(hide yes)
+			(show_name no)
+			(do_not_autoplace no)
+			(effects
+				(font
+					(size 1.27 1.27)
+				)
+			)
+		)
+		(property "LCSC Part Number" "C3819527"
 			(at 212.09 100.33 0)
 			(hide yes)
@@
 			)
 		)
-		(property "LCSC_Part_Number" "C14663"
-			(at 143.51 64.77 0)
-			(hide yes)
-			(show_name no)
-			(do_not_autoplace no)
-			(effects
-				(font
-					(size 1.27 1.27)
-				)
-			)
-		)
 		(property "Availability" ""
 			(at 143.51 64.77 0)
@@
 		)
 		(property "SnapEDA_Link" ""
+			(at 143.51 64.77 0)
+			(hide yes)
+			(show_name no)
+			(do_not_autoplace no)
+			(effects
+				(font
+					(size 1.27 1.27)
+				)
+			)
+		)
+		(property "LCSC Part Number" "C14663"
 			(at 143.51 64.77 0)
 			(hide yes)
@@
 			)
 		)
-		(property "LCSC_Part_Number" "C77093"
-			(at 160.02 64.77 0)
-			(hide yes)
-			(show_name no)
-			(do_not_autoplace no)
-			(effects
-				(font
-					(size 1.27 1.27)
-				)
-			)
-		)
 		(property "Availability" ""
 			(at 160.02 64.77 0)
@@
 		)
 		(property "SnapEDA_Link" ""
+			(at 160.02 64.77 0)
+			(hide yes)
+			(show_name no)
+			(do_not_autoplace no)
+			(effects
+				(font
+					(size 1.27 1.27)
+				)
+			)
+		)
+		(property "LCSC Part Number" "C14860"
 			(at 160.02 64.77 0)
 			(hide yes)
@@
 			)
 		)
-		(property "LCSC_Part_Number" "C910544"
-			(at 149.86 105.41 0)
-			(hide yes)
-			(show_name no)
-			(do_not_autoplace no)
-			(effects
-				(font
-					(size 1.27 1.27)
-				)
-			)
-		)
 		(property "Availability" ""
 			(at 149.86 105.41 0)
@@
 		)
 		(property "SnapEDA_Link" ""
+			(at 149.86 105.41 0)
+			(hide yes)
+			(show_name no)
+			(do_not_autoplace no)
+			(effects
+				(font
+					(size 1.27 1.27)
+				)
+			)
+		)
+		(property "LCSC Part Number" "C910544"
 			(at 149.86 105.41 0)
 			(hide yes)
@@
 			)
 		)
-		(property "LCSC_Part_Number" "C85840"
-			(at 177.8 91.44 0)
-			(hide yes)
-			(show_name no)
-			(do_not_autoplace no)
-			(effects
-				(font
-					(size 1.27 1.27)
-				)
-			)
-		)
 		(property "Availability" ""
 			(at 177.8 91.44 90)
@@
 		)
 		(property "SnapEDA_Link" ""
+			(at 177.8 91.44 90)
+			(hide yes)
+			(show_name no)
+			(do_not_autoplace no)
+			(effects
+				(font
+					(size 1.27 1.27)
+				)
+			)
+		)
+		(property "LCSC Part Number" "C85840"
 			(at 177.8 91.44 90)
 			(hide yes)
@@
 			)
 		)
-		(property "LCSC_Part_Number" "C1588"
-			(at 193.04 101.6 0)
-			(hide yes)
-			(show_name no)
-			(do_not_autoplace no)
-			(effects
-				(font
-					(size 1.27 1.27)
-				)
-			)
-		)
 		(property "Availability" ""
 			(at 193.04 101.6 0)
@@
 		)
 		(property "SnapEDA_Link" ""
+			(at 193.04 101.6 0)
+			(hide yes)
+			(show_name no)
+			(do_not_autoplace no)
+			(effects
+				(font
+					(size 1.27 1.27)
+				)
+			)
+		)
+		(property "LCSC Part Number" "C1588"
 			(at 193.04 101.6 0)
 			(hide yes)
@@
 			)
 		)
-		(property "LCSC_Part_Number" "C85840"
-			(at 177.8 106.68 0)
-			(hide yes)
-			(show_name no)
-			(do_not_autoplace no)
-			(effects
-				(font
-					(size 1.27 1.27)
-				)
-			)
-		)
 		(property "Availability" ""
 			(at 177.8 106.68 90)
@@
 			(at 177.8 106.68 90)
 			(hide yes)
+			(show_name no)
+			(do_not_autoplace no)
+			(effects
+				(font
+					(size 1.27 1.27)
+				)
+			)
+		)
+		(property "LCSC Part Number" "C85840"
+			(at 177.8 106.68 90)
+			(hide yes)

Commit message: Cost reductions for JCLPCB
Parts:
- removed H12: Conn_01x02, TerminalBlock_Phoenix:TerminalBlock_Phoenix_PT-1,5-2-3.5-H_1x02_P3.50mm_Horizontal, symbol Connector_Generic:Conn_01x02
- added U7: KF350-3.5-2P, easyeda2kicad:CONN-TH_P3.50_KF350-3.5-2P, symbol easyeda2kicad:KF350-3.5-2P
- C2: LCSC Part Number C14860 -> C13585
Connections:
- net at C3.1, FB1.2: now also U7.2
- net at C4.2, FB2.2: now also U7.1
Changed lines of the file:
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@@
-	(wire
-		(pts
-			(xy 207.01 91.44) (xy 207.01 97.79)
-		)
-		(stroke
-			(width 0)
-			(type default)
-		)
-	)
 	(wire
 		(pts
@@
 	(wire
 		(pts
-			(xy 193.04 106.68) (xy 207.01 106.68)
-		)
-		(stroke
-			(width 0)
-			(type default)
-		)
-	)
-	(wire
-		(pts
-			(xy 187.96 91.44) (xy 207.01 91.44)
+			(xy 193.04 106.68) (xy 214.63 106.68)
+		)
+		(stroke
+			(width 0)
+			(type default)
+		)
+	)
+	(wire
+		(pts
+			(xy 187.96 91.44) (xy 214.63 91.44)
 		)
 		(stroke
@@
 	(wire
 		(pts
+			(xy 214.63 91.44) (xy 214.63 97.79)
+		)
+		(stroke
+			(width 0)
+			(type default)
+		)
+	)
+	(wire
+		(pts
 			(xy 165.1 97.79) (xy 162.56 97.79)
 		)
@@
 	(wire
 		(pts
-			(xy 207.01 100.33) (xy 207.01 106.68)
+			(xy 214.63 100.33) (xy 214.63 106.68)
 		)
 		(stroke
@@
 	)
 	(symbol
-		(lib_id "Connector_Generic:Conn_01x02")
-		(at 212.09 100.33 0)
-		(mirror x)
-		(unit 1)
-		(body_style 1)
-		(exclude_from_sim no)
-		(in_bom yes)
-		(on_board yes)
-		(in_pos_files yes)
-		(dnp no)
-		(property "Reference" "H12"
-			(at 214.63 100.3301 0)
-			(show_name no)
-			(do_not_autoplace no)
-			(effects
-				(font
-					(size 1.27 1.27)
-				)
-				(justify left)
-			)
-		)
-		(property "Value" "Conn_01x02"
-			(at 214.63 97.7901 0)
-			(show_name no)
-			(do_not_autoplace no)
-			(effects
-				(font
-					(size 1.27 1.27)
-				)
-				(justify left)
-			)
-		)
-		(property "Footprint" "TerminalBlock_Phoenix:TerminalBlock_Phoenix_PT-1,5-2-3.5-H_1x02_P3.50mm_Horizontal"
-			(at 212.09 100.33 0)
-			(hide yes)
-			(show_name no)
-			(do_not_autoplace no)
-			(effects
-				(font
-					(size 1.27 1.27)
-				)
-			)
-		)
-		(property "Datasheet" ""
-			(at 212.09 100.33 0)
-			(hide yes)
-			(show_name no)
-			(do_not_autoplace no)
-			(effects
-				(font
-					(size 1.27 1.27)
-				)
-			)
-		)
-		(property "Description" "Generic connector, single row, 01x02, script generated (kicad-library-utils/schlib/autogen/connector/)"
-			(at 212.09 100.33 0)
-			(hide yes)
-			(show_name no)
-			(do_not_autoplace no)
-			(effects
-				(font
-					(size 1.27 1.27)
-				)
-			)
-		)
-		(property "Manufacturer_Part_Number" "1984617"
-			(at 212.09 100.33 0)
-			(hide yes)
-			(show_name no)
-			(do_not_autoplace no)
-			(effects
-				(font
-					(size 1.27 1.27)
-				)
-			)
-		)
-		(property "Availability" ""
-			(at 212.09 100.33 0)
-			(hide yes)
-			(show_name no)
-			(do_not_autoplace no)
-			(effects
-				(font
-					(size 1.27 1.27)
-				)
-			)
-		)
-		(property "Check_prices" ""
-			(at 212.09 100.33 0)
-			(hide yes)
-			(show_name no)
-			(do_not_autoplace no)
-			(effects
-				(font
-					(size 1.27 1.27)
-				)
-			)
-		)
-		(property "Comment" ""
-			(at 212.09 100.33 0)
-			(hide yes)
-			(show_name no)
-			(do_not_autoplace no)
-			(effects
-				(font
-					(size 1.27 1.27)
-				)
-			)
-		)
-		(property "EU_RoHS_Compliance" ""
-			(at 212.09 100.33 0)
-			(hide yes)
-			(show_name no)
-			(do_not_autoplace no)
-			(effects
-				(font
-					(size 1.27 1.27)
-				)
-			)
-		)
-		(property "MF" ""
-			(at 212.09 100.33 0)
-			(hide yes)
-			(show_name no)
-			(do_not_autoplace no)
-			(effects
-				(font
-					(size 1.27 1.27)
-				)
-			)
-		)
-		(property "MP" ""
-			(at 212.09 100.33 0)
-			(hide yes)
-			(show_name no)
-			(do_not_autoplace no)
-			(effects
-				(font
-					(size 1.27 1.27)
-				)
-			)
-		)
-		(property "PARTREV" ""
-			(at 212.09 100.33 0)
-			(hide yes)
-			(show_name no)
-			(do_not_autoplace no)
-			(effects
-				(font
-					(size 1.27 1.27)
-				)
-			)
-		)
-		(property "Package" ""
-			(at 212.09 100.33 0)
-			(hide yes)
-			(show_name no)
-			(do_not_autoplace no)
-			(effects
-				(font
-					(size 1.27 1.27)
-				)
-			)
-		)
-		(property "Price" ""
-			(at 212.09 100.33 0)
-			(hide yes)
-			(show_name no)
-			(do_not_autoplace no)
-			(effects
-				(font
-					(size 1.27 1.27)
-				)
-			)
-		)
-		(property "Purchase-URL" ""
-			(at 212.09 100.33 0)
-			(hide yes)
-			(show_name no)
-			(do_not_autoplace no)
-			(effects
-				(font
-					(size 1.27 1.27)
-				)
-			)
-		)
-		(property "STANDARD" ""
-			(at 212.09 100.33 0)
-			(hide yes)
-			(show_name no)
-			(do_not_autoplace no)
-			(effects
-				(font
-					(size 1.27 1.27)
-				)
-			)
-		)
-		(property "SnapEDA_Link" ""
-			(at 212.09 100.33 0)
-			(hide yes)
-			(show_name no)
-			(do_not_autoplace no)
-			(effects
-				(font
-					(size 1.27 1.27)
-				)
-			)
-		)
-		(property "LCSC Part Number" "C3819527"
-			(at 212.09 100.33 0)
-			(hide yes)
-			(show_name no)
-			(do_not_autoplace no)
-			(effects
-				(font
-					(size 1.27 1.27)
-				)
-			)
-		)
-		(pin "1"
-		)
-		(pin "2"
-		)
-		(instances
-			(project "HDD Synth Prototype MK5"
-				(path "/1a22431a-ba36-40a0-9a7e-c2a82ec69c53/2950dfc3-c685-4e23-94aa-d1af22619645"
-					(reference "H12")
-					(unit 1)
-				)
-			)
-			(project "HDD Synth prototype MK3"
-				(path "/5a2f0aa7-670f-4d0d-8d56-ad98c847383a/a3500c8b-1cb4-4280-8b2f-37934c522aa7"
-					(reference "H6")
-					(unit 1)
-				)
-			)
-			(project "FDD Synth prototype MK1"
-				(path "/ed113b11-1722-4efb-9669-9e8c19f5c8fd/ceef9c1f-e4ce-45b2-b9fe-22340e8232b8"
-					(reference "H6")
-					(unit 1)
-				)
-			)
-		)
-	)
-	(symbol
 		(lib_id "Device:C")
 		(at 143.51 64.77 180)
@@
 			)
 		)
-		(property "LCSC Part Number" "C14860"
+		(property "LCSC Part Number" "C13585"
 			(at 160.02 64.77 0)
 			(hide yes)
@@
 					(unit 1)
 				)
+			)
+		)
+	)
+	(symbol
+		(lib_id "easyeda2kicad:KF350-3.5-2P")
+		(at 210.82 99.06 180)
+		(unit 1)
+		(body_style 1)
+		(exclude_from_sim no)
+		(in_bom yes)
+		(on_board yes)
+		(in_pos_files yes)
+		(dnp no)
+		(fields_autoplaced yes)
+		(property "Reference" "U7"
+			(at 209.55 90.17 0)
+			(show_name no)
+			(do_not_autoplace no)
+			(effects
+				(font
+					(size 1.27 1.27)
+				)
+			)
+		)
+		(property "Value" "KF350-3.5-2P"
+			(at 209.55 92.71 0)
+			(show_name no)
+			(do_not_autoplace no)
+			(effects
+				(font
+					(size 1.27 1.27)
+				)
+			)
+		)
+		(property "Footprint" "easyeda2kicad:CONN-TH_P3.50_KF350-3.5-2P"
+			(at 210.82 90.17 0)
+			(hide yes)
+			(show_name no)
+			(do_not_autoplace no)
+			(effects
+				(font
+					(size 1.27 1.27)
+				)
+			)
+		)
+		(property "Datasheet" "https://lcsc.com/product-detail/New-Quadratic-Unclassified-Data_Cixi-Kefa-Elec-KF350-3-5-2P_C474892.html"
+			(at 210.82 87.63 0)
+			(hide yes)
+			(show_name no)
+			(do_not_autoplace no)
+			(effects
+				(font
+					(size 1.27 1.27)
+				)
+			)
+		)
+		(property "Description" ""
+			(at 210.82 99.06 0)
+			(hide yes)
+			(show_name no)
+			(do_not_autoplace no)
+			(effects
+				(font
+					(size 1.27 1.27)
+				)
+			)
+		)
+		(property "Manufacturer" "KEFA(科发)"
+			(at 210.82 85.09 0)
+			(hide yes)
+			(show_name no)
+			(do_not_autoplace no)
+			(effects
+				(font
+					(size 1.27 1.27)
+				)
+			)
+		)
+		(property "MPN" "KF350-3.5-2P"
+			(at 210.82 82.55 0)
+			(hide yes)
+			(show_name no)
+			(do_not_autoplace no)
+			(effects
+				(font
+					(size 1.27 1.27)
+				)
+			)
+		)
+		(property "LCSC Part" "C474892"
+			(at 210.82 80.01 0)
+			(hide yes)
+			(show_name no)
+			(do_not_autoplace no)
+			(effects
+				(font
+					(size 1.27 1.27)
+				)
+			)
+		)
+		(pin "1"
+		)
+		(pin "2"
+		)
+		(instances
+			(project "HDD Synth Prototype MK5"
+				(path "/1a22431a-ba36-40a0-9a7e-c2a82ec69c53/2950dfc3-c685-4e23-94aa-d1af22619645"
+					(reference "U7")
+					(unit 1)
+				)

Commit message: Tweaks
Connections:
- net POWER_5V_SUP: no longer U2.2 (GAIN_SLOT)
- new net VSYS: U2.2 (GAIN_SLOT)
Changed lines of the file:
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@@
 	(wire
 		(pts
-			(xy 121.92 110.49) (xy 137.16 110.49)
+			(xy 102.87 110.49) (xy 137.16 110.49)
 		)
 		(stroke
@@
 		)
 	)
-	(global_label "POWER_5V_SUP"
+	(global_label "VSYS"
 		(shape bidirectional)
-		(at 121.92 110.49 180)
+		(at 102.87 110.49 180)
 		(fields_autoplaced yes)
 		(effects
@@
 		)
 		(property "Intersheetrefs" "${INTERSHEET_REFS}"
-			(at 103.3093 110.49 0)
+			(at 94.1773 110.49 0)
 			(hide yes)
 			(show_name no)

Commit message: Tweaks
Connections:
- net POWER_5V_SUP is gone; now on net VSYS: C1.2, C2.2, U2.7 (VDD), U2.8 (VDD)
Changed lines of the file:
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@@
 		)
 	)
-	(global_label "POWER_5V_SUP"
+	(global_label "VSYS"
 		(shape bidirectional)
 		(at 149.86 55.88 90)
@@
 		)
 		(property "Intersheetrefs" "${INTERSHEET_REFS}"
-			(at 149.86 37.2693 90)
+			(at 149.86 47.1873 90)
 			(hide yes)
 			(show_name no)

Commit message: 5.3.0 sent to JCLPCB
Parts:
- U7: LCSC Part C474892 -> (none); LCSC Part Number (none) -> C474892
Changed lines of the file:
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@@
 			)
 		)
-		(property "LCSC Part" "C474892"
+		(property "LCSC Part" ""
 			(at 210.82 80.01 0)
 			(hide yes)
 			(show_name no)
+			(do_not_autoplace no)
+			(effects
+				(font
+					(size 1.27 1.27)
+				)
+			)
+		)
+		(property "LCSC Part Number" "C474892"
+			(at 210.82 99.06 0)
+			(hide yes)
+			(show_name no)
