File: 2_prototype_mk5/slot_adapters/isa/HDD Synth ISA adapter.kicad_sch (KiCad schematic)
At the start: 8 parts, among them J1 Conn_01x02_Socket, J2 Conn_01x05_Socket, J3 Bus_ISA_8bit, J4 Conn_01x02_Socket, SW1 SW_Push, SW2 PEC12R-2120F-S0012

Commit message: MK5 revision 2 hardware updates and ISA adapter revisions
Ignore VSCode local-history artifacts going forward.

Co-Authored-By: Claude Sonnet 5 <noreply@anthropic.com>
Parts:
- added J5, J6, J7, J8: Conn_01x02_Socket, Connector_PinSocket_2.54mm:PinSocket_1x02_P2.54mm_Vertical, symbol Connector:Conn_01x02_Socket
Connections:
- new net: J5.1 (Pin_1), J6.1 (Pin_1)
- new net: J5.2 (Pin_2), J6.2 (Pin_2)
- new net: J7.1 (Pin_1), J8.1 (Pin_1)
- new net: J7.2 (Pin_2), J8.2 (Pin_2)
Other:
- note added: "LED in"
- note added: "LED out"
